Commit message: fix: export changes to URDF

File: deep_ballbot_description/urdf/deep_ballbot.xacro (robot description, xacro)
@@ -64,4 +64,24 @@
   </collision>
 </link>
+<link name="base_shell3_1">
+  <inertial>
+    <origin rpy="0 0 0" xyz="0.0315493029461081 0.01821499854867909 0.021364464404157207"/>
+    <mass value="0.03897424370875779"/>
+    <inertia ixx="3.3e-05" ixy="1.1e-05" ixz="-6e-06" iyy="2e-05" iyz="-3e-06" izz="3.8e-05"/>
+  </inertial>
+  <visual>
+    <origin rpy="0 0 0" xyz="-0.0 -0.0 -0.139"/>
+    <geometry>
+      <mesh filename="package://deep_ballbot_description/meshes/base_shell3_1.stl" scale="0.001 0.001 0.001"/>
+    </geometry>
+    <material name="silver"/>
+  </visual>
+  <collision>
+    <origin rpy="0 0 0" xyz="-0.0 -0.0 -0.139"/>
+    <geometry>
+      <mesh filename="package://deep_ballbot_description/meshes/base_shell3_1.stl" scale="0.001 0.001 0.001"/>
+    </geometry>
+  </collision>
+</link>
 <link name="base_plate2_1">
   <inertial>
@@ -84,24 +104,4 @@
   </collision>
 </link>
-<link name="base_plate2_1">
-  <inertial>
-    <origin rpy="0 0 0" xyz="-0.026715575075313323 -0.005670206030594099 0.0029137797806522425"/>
-    <mass value="0.029331775102842923"/>
-    <inertia ixx="1.5e-05" ixy="-6e-06" ixz="-0.0" iyy="9e-06" iyz="0.0" izz="2.4e-05"/>
-  </inertial>
-  <visual>
-    <origin rpy="0 0 0" xyz="-0.059036 0.01299 -0.184"/>
-    <geometry>
-      <mesh filename="package://deep_ballbot_description/meshes/base_plate2_1.stl" scale="0.001 0.001 0.001"/>
-    </geometry>
-    <material name="silver"/>
-  </visual>
-  <collision>
-    <origin rpy="0 0 0" xyz="-0.059036 0.01299 -0.184"/>
-    <geometry>
-      <mesh filename="package://deep_ballbot_description/meshes/base_plate2_1.stl" scale="0.001 0.001 0.001"/>
-    </geometry>
-  </collision>
-</link>
 <link name="base_plate3_1">
   <inertial>
@@ -124,21 +124,1261 @@
   </collision>
 </link>
-<link name="base_plate3_1">
-  <inertial>
-    <origin rpy="0 0 0" xyz="0.018268000000002907 -0.02030158793881661 0.002913779780652437"/>
-    <mass value="0.029331775102842902"/>
-    <inertia ixx="5e-06" ixy="-0.0" ixz="0.0" iyy="1.9e-05" iyz="-0.0" izz="2.4e-05"/>
-  </inertial>
-  <visual>
-    <origin rpy="0 0 0" xyz="0.018268 -0.057622 -0.184"/>
-    <geometry>
-      <mesh filename="package://deep_ballbot_description/meshes/base_plate3_1.stl" scale="0.001 0.001 0.001"/>
-    </geometry>
-    <material name="silver"/>
-  </visual>
-  <collision>
-    <origin rpy="0 0 0" xyz="0.018268 -0.057622 -0.184"/>
-    <geometry>
-      <mesh filename="package://deep_ballbot_description/meshes/base_plate3_1.stl" scale="0.001 0.001 0.001"/>
+<link name="vertical_bay1_1">
+  <inertial>
+    <origin rpy="0 0 0" xyz="-1.6167557852567183e-07 1.1086679559124679e-07 0.03426796949760952"/>
+    <mass value="0.02673500652833671"/>
+    <inertia ixx="1.7e-05" ixy="4e-06" ixz="0.0" iyy="1.3e-05" iyz="0.0" izz="8e-06"/>
+  </inertial>
+  <visual>
+    <origin rpy="0 0 0" xyz="0.023921 0.013811 -0.187"/>
+    <geometry>
+      <mesh filename="package://deep_ballbot_description/meshes/vertical_bay1_1.stl" scale="0.001 0.001 0.001"/>
+    </geometry>
+    <material name="silver"/>
+  </visual>
+  <collision>
+    <origin rpy="0 0 0" xyz="0.023921 0.013811 -0.187"/>
+    <geometry>
+      <mesh filename="package://deep_ballbot_description/meshes/vertical_bay1_1.stl" scale="0.001 0.001 0.001"/>
+    </geometry>
+  </collision>
+</link>
+<link name="vertical_bay2_1">
+  <inertial>
+    <origin rpy="0 0 0" xyz="1.6167524612489825e-07 1.108674625403816e-07 0.034307521329889706"/>
+    <mass value="0.026769047843990496"/>
+    <inertia ixx="1.8e-05" ixy="-4e-06" ixz="0.0" iyy="1.3e-05" iyz="-0.0" izz="8e-06"/>
+  </inertial>
+  <visual>
+    <origin rpy="0 0 0" xyz="-0.023921 0.013811 -0.187"/>
+    <geometry>
+      <mesh filename="package://deep_ballbot_description/meshes/vertical_bay2_1.stl" scale="0.001 0.001 0.001"/>
+    </geometry>
+    <material name="silver"/>
+  </visual>
+  <collision>
+    <origin rpy="0 0 0" xyz="-0.023921 0.013811 -0.187"/>
+    <geometry>
+      <mesh filename="package://deep_ballbot_description/meshes/vertical_bay2_1.stl" scale="0.001 0.001 0.001"/>
+    </geometry>
+  </collision>
+</link>
+<link name="vertical_bay3_1">
+  <inertial>
+    <origin rpy="0 0 0" xyz="4.8585964403268e-15 -2.2173493367805275e-07 0.03430752132988982"/>
+    <mass value="0.026769047843990493"/>
+    <inertia ixx="1.1e-05" ixy="-0.0" ixz="-0.0" iyy="2e-05" iyz="0.0" izz="8e-06"/>
+  </inertial>
+  <visual>
+    <origin rpy="0 0 0" xyz="-0.0 -0.027622 -0.187"/>
+    <geometry>
+      <mesh filename="package://deep_ballbot_description/meshes/vertical_bay3_1.stl" scale="0.001 0.001 0.001"/>
+    </geometry>
+    <material name="silver"/>
+  </visual>
+  <collision>
+    <origin rpy="0 0 0" xyz="-0.0 -0.027622 -0.187"/>
+    <geometry>
+      <mesh filename="package://deep_ballbot_description/meshes/vertical_bay3_1.stl" scale="0.001 0.001 0.001"/>
+    </geometry>
+  </collision>
+</link>
+<link name="breadboard_1">
+  <inertial>
+    <origin rpy="0 0 0" xyz="-3.512780628184276e-10 0.017499602320883354 0.003999999999999948"/>
+    <mass value="0.016254000000000088"/>
+    <inertia ixx="2e-06" ixy="-0.0" ixz="-0.0" iyy="3e-06" iyz="0.0" izz="4e-06"/>
+  </inertial>
+  <visual>
+    <origin rpy="0 0 0" xyz="0.0 0.047631 -0.258"/>
+    <geometry>
+      <mesh filename="package://deep_ballbot_description/meshes/breadboard_1.stl" scale="0.001 0.001 0.001"/>
+    </geometry>
+    <material name="silver"/>
+  </visual>
+  <collision>
+    <origin rpy="0 0 0" xyz="0.0 0.047631 -0.258"/>
+    <geometry>
+      <mesh filename="package://deep_ballbot_description/meshes/breadboard_1.stl" scale="0.001 0.001 0.001"/>
+    </geometry>
+  </collision>
+</link>
+<link name="arduino_nano_1">
+  <inertial>
+    <origin rpy="0 0 0" xyz="-0.0015922703223249265 0.0015396023112441357 0.014355883406889147"/>
+    <mass value="0.014605507737955568"/>
+    <inertia ixx="1e-06" ixy="-0.0" ixz="0.0" iyy="2e-06" iyz="0.0" izz="3e-06"/>
+  </inertial>
+  <visual>
+    <origin rpy="0 0 0" xyz="-0.000352 0.031671 -0.255"/>
+    <geometry>
+      <mesh filename="package://deep_ballbot_description/meshes/arduino_nano_1.stl" scale="0.001 0.001 0.001"/>
+    </geometry>
+    <material name="silver"/>
+  </visual>
+  <collision>
+    <origin rpy="0 0 0" xyz="-0.000352 0.031671 -0.255"/>
+    <geometry>
+      <mesh filename="package://deep_ballbot_description/meshes/arduino_nano_1.stl" scale="0.001 0.001 0.001"/>
+    </geometry>
+  </collision>
+</link>
+<link name="rasbperry_pi_1">
+  <inertial>
+    <origin rpy="0 0 0" xyz="-0.0012540090701389588 0.004888830200196736 0.057465472519733274"/>
+    <mass value="0.13472167579144456"/>
+    <inertia ixx="8.3e-05" ixy="0.0" ixz="-0.0" iyy="0.000118" iyz="-9e-06" izz="4.1e-05"/>
+  </inertial>
+  <visual>
+    <origin rpy="0 0 0" xyz="0.0 -0.0105 -0.258"/>
+    <geometry>
+      <mesh filename="package://deep_ballbot_description/meshes/rasbperry_pi_1.stl" scale="0.001 0.001 0.001"/>
+    </geometry>
+    <material name="silver"/>
+  </visual>
+  <collision>
+    <origin rpy="0 0 0" xyz="0.0 -0.0105 -0.258"/>
+    <geometry>
+      <mesh filename="package://deep_ballbot_description/meshes/rasbperry_pi_1.stl" scale="0.001 0.001 0.001"/>
+    </geometry>
+  </collision>
+</link>
+<link name="motor_mount1_1">
+  <inertial>
+    <origin rpy="0 0 0" xyz="0.008784093083896216 -0.005071216542772684 -0.01575982915390231"/>
+    <mass value="0.08608420182582005"/>
+    <inertia ixx="3.8e-05" ixy="-9e-06" ixz="1e-05" iyy="2.8e-05" iyz="-6e-06" izz="4.3e-05"/>
+  </inertial>
+  <visual>
+    <origin rpy="0 0 0" xyz="0.046487 -0.026839 -0.171056"/>
+    <geometry>
+      <mesh filename="package://deep_ballbot_description/meshes/motor_mount1_1.stl" scale="0.001 0.001 0.001"/>
+    </geometry>
+    <material name="silver"/>
+  </visual>
+  <collision>
+    <origin rpy="0 0 0" xyz="0.046487 -0.026839 -0.171056"/>
+    <geometry>
+      <mesh filename="package://deep_ballbot_description/meshes/motor_mount1_1.stl" scale="0.001 0.001 0.001"/>
+    </geometry>
+  </collision>
+</link>
+<link name="motor_mount2_1">
+  <inertial>
+    <origin rpy="0 0 0" xyz="1.2758713609389452e-14 0.010142433085668257 -0.01575982915375221"/>
+    <mass value="0.08608420182581958"/>
+    <inertia ixx="2.3e-05" ixy="0.0" ixz="-0.0" iyy="4.3e-05" iyz="1.1e-05" izz="4.3e-05"/>
+  </inertial>
+  <visual>
+    <origin rpy="0 0 0" xyz="-0.0 0.053678 -0.171056"/>
+    <geometry>
+      <mesh filename="package://deep_ballbot_description/meshes/motor_mount2_1.stl" scale="0.001 0.001 0.001"/>
+    </geometry>
+    <material name="silver"/>
+  </visual>
+  <collision>
+    <origin rpy="0 0 0" xyz="-0.0 0.053678 -0.171056"/>
+    <geometry>
+      <mesh filename="package://deep_ballbot_description/meshes/motor_mount2_1.stl" scale="0.001 0.001 0.001"/>
+    </geometry>
+  </collision>
+</link>
+<link name="motor_mount3_1">
+  <inertial>
+    <origin rpy="0 0 0" xyz="-0.008784093083910476 -0.005071216542747357 -0.015759829153902005"/>
+    <mass value="0.08608420182581962"/>
+    <inertia ixx="3.8e-05" ixy="9e-06" ixz="-1e-05" iyy="2.8e-05" iyz="-6e-06" izz="4.3e-05"/>
+  </inertial>
+  <visual>
+    <origin rpy="0 0 0" xyz="-0.046487 -0.026839 -0.171056"/>
+    <geometry>
+      <mesh filename="package://deep_ballbot_description/meshes/motor_mount3_1.stl" scale="0.001 0.001 0.001"/>
+    </geometry>
+    <material name="silver"/>
+  </visual>
+  <collision>
+    <origin rpy="0 0 0" xyz="-0.046487 -0.026839 -0.171056"/>
+    <geometry>
+      <mesh filename="package://deep_ballbot_description/meshes/motor_mount3_1.stl" scale="0.001 0.001 0.001"/>
+    </geometry>
+  </collision>
+</link>
+<link name="arduino_mount1_1">
+  <inertial>
+    <origin rpy="0 0 0" xyz="-0.0017985403607222034 -0.0017781689855505562 -2.1615661864288205e-05"/>
+    <mass value="0.023201510107992093"/>
+    <inertia ixx="1.3e-05" ixy="5e-06" ixz="-0.0" iyy="8e-06" iyz="0.0" izz="1.2e-05"/>
+  </inertial>
+  <visual>
+    <origin rpy="0 0 0" xyz="0.026519 0.015311 -0.2195"/>
+    <geometry>
+      <mesh filename="package://deep_ballbot_description/meshes/arduino_mount1_1.stl" scale="0.001 0.001 0.001"/>
+    </geometry>
+    <material name="silver"/>
+  </visual>
+  <collision>
+    <origin rpy="0 0 0" xyz="0.026519 0.015311 -0.2195"/>
+    <geometry>
+      <mesh filename="package://deep_ballbot_description/meshes/arduino_mount1_1.stl" scale="0.001 0.001 0.001"/>
+    </geometry>
+  </collision>
+</link>
+<link name="arduino_mount2_1">
+  <inertial>
+    <origin rpy="0 0 0" xyz="0.0024394246518729297 -0.0006681248315038978 -2.1615661864288205e-05"/>
+    <mass value="0.023201510107960607"/>
+    <inertia ixx="1.3e-05" ixy="-5e-06" ixz="-0.0" iyy="8e-06" iyz="-0.0" izz="1.2e-05"/>
+  </inertial>
+  <visual>
+    <origin rpy="0 0 0" xyz="-0.026519 0.015311 -0.2195"/>
+    <geometry>
+      <mesh filename="package://deep_ballbot_description/meshes/arduino_mount2_1.stl" scale="0.001 0.001 0.001"/>
+    </geometry>
+    <material name="silver"/>
+  </visual>
+  <collision>
+    <origin rpy="0 0 0" xyz="-0.026519 0.015311 -0.2195"/>
+    <geometry>
+      <mesh filename="package://deep_ballbot_description/meshes/arduino_mount2_1.stl" scale="0.001 0.001 0.001"/>
+    </geometry>
+  </collision>
+</link>
+<link name="arduino_mount3_1">
+  <inertial>
+    <origin rpy="0 0 0" xyz="-0.0006408842911585192 0.0024462938179583525 -2.1615661864482494e-05"/>
+    <mass value="0.023201510107976293"/>
+    <inertia ixx="5e-06" ixy="0.0" ixz="0.0" iyy="1.6e-05" iyz="0.0" izz="1.2e-05"/>
+  </inertial>
+  <visual>
+    <origin rpy="0 0 0" xyz="-0.0 -0.030622 -0.2195"/>
+    <geometry>
+      <mesh filename="package://deep_ballbot_description/meshes/arduino_mount3_1.stl" scale="0.001 0.001 0.001"/>
+    </geometry>
+    <material name="silver"/>
+  </visual>
+  <collision>
+    <origin rpy="0 0 0" xyz="-0.0 -0.030622 -0.2195"/>
+    <geometry>
+      <mesh filename="package://deep_ballbot_description/meshes/arduino_mount3_1.stl" scale="0.001 0.001 0.001"/>
+    </geometry>
+  </collision>
+</link>
+<link name="arduino1_1">
+  <inertial>
+    <origin rpy="0 0 0" xyz="0.01666958536509317 -0.034661355386450377 0.00875853373784699"/>
+    <mass value="0.0763619336554754"/>
+    <inertia ixx="4.9e-05" ixy="1.4e-05" ixz="0.0" iyy="2.9e-05" iyz="-1e-06" izz="3.5e-05"/>
+  </inertial>
+  <visual>
+    <origin rpy="0 0 0" xyz="0.047078 -0.010299 -0.211"/>
+    <geometry>
+      <mesh filename="package://deep_ballbot_description/meshes/arduino1_1.stl" scale="0.001 0.001 0.001"/>
+    </geometry>
+    <material name="silver"/>
+  </visual>
+  <collision>
+    <origin rpy="0 0 0" xyz="0.047078 -0.010299 -0.211"/>
+    <geometry>
+      <mesh filename="package://deep_ballbot_description/meshes/arduino1_1.stl" scale="0.001 0.001 0.001"/>
+    </geometry>
+  </collision>
+</link>
+<link name="arduino2_1">
+  <inertial>
+    <origin rpy="0 0 0" xyz="0.021682625979238306 0.03176671812995284 0.008758533737850571"/>
+    <mass value="0.07636193365547596"/>
+    <inertia ixx="4.6e-05" ixy="-1.6e-05" ixz="1e-06" iyy="3.2e-05" iyz="1e-06" izz="3.5e-05"/>
+  </inertial>
+  <visual>
+    <origin rpy="0 0 0" xyz="-0.01462 0.04592 -0.211"/>
+    <geometry>
+      <mesh filename="package://deep_ballbot_description/meshes/arduino2_1.stl" scale="0.001 0.001 0.001"/>
+    </geometry>
+    <material name="silver"/>
+  </visual>
+  <collision>
+    <origin rpy="0 0 0" xyz="-0.01462 0.04592 -0.211"/>
+    <geometry>
+      <mesh filename="package://deep_ballbot_description/meshes/arduino2_1.stl" scale="0.001 0.001 0.001"/>
+    </geometry>
+  </collision>
+</link>
+<link name="arduino3_1">
+  <inertial>
+    <origin rpy="0 0 0" xyz="-0.03835221134344281 0.0028936372564971197 0.008758533737798002"/>
+    <mass value="0.07636193365547513"/>
+    <inertia ixx="2.2e-05" ixy="2e-06" ixz="-1e-06" iyy="5.6e-05" iyz="0.0" izz="3.5e-05"/>
+  </inertial>
+  <visual>
+    <origin rpy="0 0 0" xyz="-0.032458 -0.035622 -0.211"/>
+    <geometry>
+      <mesh filename="package://deep_ballbot_description/meshes/arduino3_1.stl" scale="0.001 0.001 0.001"/>
+    </geometry>
+    <material name="silver"/>
+  </visual>
+  <collision>
+    <origin rpy="0 0 0" xyz="-0.032458 -0.035622 -0.211"/>
+    <geometry>
+      <mesh filename="package://deep_ballbot_description/meshes/arduino3_1.stl" scale="0.001 0.001 0.001"/>
+    </geometry>
+  </collision>
+</link>
+<link name="motor_stator1_1">
+  <inertial>
+    <origin rpy="0 0 0" xyz="0.013066369938678046 -0.007543151268848507 -0.016105881234575237"/>
+    <mass value="0.2071891794839974"/>
+    <inertia ixx="5.6e-05" ixy="-8e-06" ixz="1.6e-05" iyy="4.7e-05" iyz="-9e-06" izz="6.1e-05"/>
+  </inertial>
+  <visual>
+    <origin rpy="0 0 0" xyz="0.051386 -0.029667 -0.165399"/>
+    <geometry>
+      <mesh filename="package://deep_ballbot_description/meshes/motor_stator1_1.stl" scale="0.001 0.001 0.001"/>
+    </geometry>
+    <material name="silver"/>
+  </visual>
+  <collision>
+    <origin rpy="0 0 0" xyz="0.051386 -0.029667 -0.165399"/>
+    <geometry>
+      <mesh filename="package://deep_ballbot_description/meshes/motor_stator1_1.stl" scale="0.001 0.001 0.001"/>
+    </geometry>
+  </collision>
+</link>
+<link name="motor_stator2_1">
+  <inertial>
+    <origin rpy="0 0 0" xyz="3.454227324397115e-17 0.015087302537697307 -0.016105881234574987"/>
+    <mass value="0.20718917948399745"/>
+    <inertia ixx="4.2e-05" ixy="0.0" ixz="-0.0" iyy="6.1e-05" iyz="1.8e-05" izz="6.1e-05"/>
+  </inertial>
+  <visual>
+    <origin rpy="0 0 0" xyz="-0.0 0.059335 -0.165399"/>
+    <geometry>
+      <mesh filename="package://deep_ballbot_description/meshes/motor_stator2_1.stl" scale="0.001 0.001 0.001"/>
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