Commit message: fix: rename wheels to fix URDF export

File: deep_ballbot_description/urdf/deep_ballbot.xacro (robot description, xacro)
@@ -604,5 +604,5 @@
   </collision>
 </link>
-<link name="wheel_roller1.2_1">
+<link name="wheel_roller1_2_1">
   <inertial>
     <origin rpy="0 0 0" xyz="1.1343589664813969e-08 -1.599636010735095e-07 -4.949366528006482e-07"/>
@@ -613,5 +613,5 @@
     <origin rpy="0 0 0" xyz="0.07833 -0.045224 -0.145601"/>
     <geometry>
-      <mesh filename="package://deep_ballbot_description/meshes/wheel_roller1.2_1.stl" scale="0.001 0.001 0.001"/>
+      <mesh filename="package://deep_ballbot_description/meshes/wheel_roller1_2_1.stl" scale="0.001 0.001 0.001"/>
     </geometry>
     <material name="silver"/>
@@ -620,9 +620,9 @@
     <origin rpy="0 0 0" xyz="0.07833 -0.045224 -0.145601"/>
     <geometry>
-      <mesh filename="package://deep_ballbot_description/meshes/wheel_roller1.2_1.stl" scale="0.001 0.001 0.001"/>
-    </geometry>
-  </collision>
-</link>
-<link name="wheel_roller1.4_1">
+      <mesh filename="package://deep_ballbot_description/meshes/wheel_roller1_2_1.stl" scale="0.001 0.001 0.001"/>
+    </geometry>
+  </collision>
+</link>
+<link name="wheel_roller1_4_1">
   <inertial>
     <origin rpy="0 0 0" xyz="0.0006668609842473416 -0.0018856180530575153 -0.0025402442651766"/>
@@ -633,5 +633,5 @@
     <origin rpy="0 0 0" xyz="0.081103 -0.03322 -0.14302"/>
     <geometry>
-      <mesh filename="package://deep_ballbot_description/meshes/wheel_roller1.4_1.stl" scale="0.001 0.001 0.001"/>
+      <mesh filename="package://deep_ballbot_description/meshes/wheel_roller1_4_1.stl" scale="0.001 0.001 0.001"/>
     </geometry>
     <material name="silver"/>
@@ -640,9 +640,9 @@
     <origin rpy="0 0 0" xyz="0.081103 -0.03322 -0.14302"/>
     <geometry>
-      <mesh filename="package://deep_ballbot_description/meshes/wheel_roller1.4_1.stl" scale="0.001 0.001 0.001"/>
-    </geometry>
-  </collision>
-</link>
-<link name="wheel_roller1.9_1">
+      <mesh filename="package://deep_ballbot_description/meshes/wheel_roller1_4_1.stl" scale="0.001 0.001 0.001"/>
+    </geometry>
+  </collision>
+</link>
+<link name="wheel_roller1_9_1">
   <inertial>
     <origin rpy="0 0 0" xyz="2.1682235341879963e-07 -4.6082259215485255e-07 -9.665432673666707e-08"/>
@@ -653,5 +653,5 @@
     <origin rpy="0 0 0" xyz="0.082135 -0.017421 -0.134994"/>
     <geometry>
-      <mesh filename="package://deep_ballbot_description/meshes/wheel_roller1.9_1.stl" scale="0.001 0.001 0.001"/>
+      <mesh filename="package://deep_ballbot_description/meshes/wheel_roller1_9_1.stl" scale="0.001 0.001 0.001"/>
     </geometry>
     <material name="silver"/>
@@ -660,9 +660,9 @@
     <origin rpy="0 0 0" xyz="0.082135 -0.017421 -0.134994"/>
     <geometry>
-      <mesh filename="package://deep_ballbot_description/meshes/wheel_roller1.9_1.stl" scale="0.001 0.001 0.001"/>
-    </geometry>
-  </collision>
-</link>
-<link name="wheel_roller1.7_1">
+      <mesh filename="package://deep_ballbot_description/meshes/wheel_roller1_9_1.stl" scale="0.001 0.001 0.001"/>
+    </geometry>
+  </collision>
+</link>
+<link name="wheel_roller1_7_1">
   <inertial>
     <origin rpy="0 0 0" xyz="1.8441455529316642e-07 7.14692537720496e-08 3.016277919237753e-07"/>
@@ -673,5 +673,5 @@
     <origin rpy="0 0 0" xyz="0.073084 -0.011884 -0.124387"/>
     <geometry>
-      <mesh filename="package://deep_ballbot_description/meshes/wheel_roller1.7_1.stl" scale="0.001 0.001 0.001"/>
+      <mesh filename="package://deep_ballbot_description/meshes/wheel_roller1_7_1.stl" scale="0.001 0.001 0.001"/>
     </geometry>
     <material name="silver"/>
@@ -680,9 +680,9 @@
     <origin rpy="0 0 0" xyz="0.073084 -0.011884 -0.124387"/>
     <geometry>
-      <mesh filename="package://deep_ballbot_description/meshes/wheel_roller1.7_1.stl" scale="0.001 0.001 0.001"/>
-    </geometry>
-  </collision>
-</link>
-<link name="wheel_roller1.12_1">
+      <mesh filename="package://deep_ballbot_description/meshes/wheel_roller1_7_1.stl" scale="0.001 0.001 0.001"/>
+    </geometry>
+  </collision>
+</link>
+<link name="wheel_roller1_12_1">
   <inertial>
     <origin rpy="0 0 0" xyz="-4.134077118272961e-07 -3.3080520738058145e-07 -1.7636573396151434e-07"/>
@@ -693,5 +693,5 @@
     <origin rpy="0 0 0" xyz="0.063771 -0.006813 -0.113787"/>
     <geometry>
-      <mesh filename="package://deep_ballbot_description/meshes/wheel_roller1.12_1.stl" scale="0.001 0.001 0.001"/>
+      <mesh filename="package://deep_ballbot_description/meshes/wheel_roller1_12_1.stl" scale="0.001 0.001 0.001"/>
     </geometry>
     <material name="silver"/>
@@ -700,9 +700,9 @@
     <origin rpy="0 0 0" xyz="0.063771 -0.006813 -0.113787"/>
     <geometry>
-      <mesh filename="package://deep_ballbot_description/meshes/wheel_roller1.12_1.stl" scale="0.001 0.001 0.001"/>
-    </geometry>
-  </collision>
-</link>
-<link name="wheel_roller1.5_1">
+      <mesh filename="package://deep_ballbot_description/meshes/wheel_roller1_12_1.stl" scale="0.001 0.001 0.001"/>
+    </geometry>
+  </collision>
+</link>
+<link name="wheel_roller1_5_1">
   <inertial>
     <origin rpy="0 0 0" xyz="4.571799286992584e-07 -4.655576237438952e-07 6.072471998852524e-08"/>
@@ -713,5 +713,5 @@
     <origin rpy="0 0 0" xyz="0.052608 -0.015208 -0.108316"/>
     <geometry>
-      <mesh filename="package://deep_ballbot_description/meshes/wheel_roller1.5_1.stl" scale="0.001 0.001 0.001"/>
+      <mesh filename="package://deep_ballbot_description/meshes/wheel_roller1_5_1.stl" scale="0.001 0.001 0.001"/>
     </geometry>
     <material name="silver"/>
@@ -720,9 +720,9 @@
     <origin rpy="0 0 0" xyz="0.052608 -0.015208 -0.108316"/>
     <geometry>
-      <mesh filename="package://deep_ballbot_description/meshes/wheel_roller1.5_1.stl" scale="0.001 0.001 0.001"/>
-    </geometry>
-  </collision>
-</link>
-<link name="wheel_roller1.10_1">
+      <mesh filename="package://deep_ballbot_description/meshes/wheel_roller1_5_1.stl" scale="0.001 0.001 0.001"/>
+    </geometry>
+  </collision>
+</link>
+<link name="wheel_roller1_10_1">
   <inertial>
     <origin rpy="0 0 0" xyz="3.574854795726501e-07 -3.6339927947381945e-07 9.819223642515418e-08"/>
@@ -733,5 +733,5 @@
     <origin rpy="0 0 0" xyz="0.041588 -0.024011 -0.103174"/>
     <geometry>
-      <mesh filename="package://deep_ballbot_description/meshes/wheel_roller1.10_1.stl" scale="0.001 0.001 0.001"/>
+      <mesh filename="package://deep_ballbot_description/meshes/wheel_roller1_10_1.stl" scale="0.001 0.001 0.001"/>
     </geometry>
     <material name="silver"/>
@@ -740,9 +740,9 @@
     <origin rpy="0 0 0" xyz="0.041588 -0.024011 -0.103174"/>
     <geometry>
-      <mesh filename="package://deep_ballbot_description/meshes/wheel_roller1.10_1.stl" scale="0.001 0.001 0.001"/>
-    </geometry>
-  </collision>
-</link>
-<link name="wheel_roller1.6_1">
+      <mesh filename="package://deep_ballbot_description/meshes/wheel_roller1_10_1.stl" scale="0.001 0.001 0.001"/>
+    </geometry>
+  </collision>
+</link>
+<link name="wheel_roller1_6_1">
   <inertial>
     <origin rpy="0 0 0" xyz="-1.5083097651413802e-07 4.335249430553745e-07 -4.748097087031722e-07"/>
@@ -753,5 +753,5 @@
     <origin rpy="0 0 0" xyz="0.039475 -0.037946 -0.108313"/>
     <geometry>
-      <mesh filename="package://deep_ballbot_description/meshes/wheel_roller1.6_1.stl" scale="0.001 0.001 0.001"/>
+      <mesh filename="package://deep_ballbot_description/meshes/wheel_roller1_6_1.stl" scale="0.001 0.001 0.001"/>
     </geometry>
     <material name="silver"/>
@@ -760,9 +760,9 @@
     <origin rpy="0 0 0" xyz="0.039475 -0.037946 -0.108313"/>
     <geometry>
-      <mesh filename="package://deep_ballbot_description/meshes/wheel_roller1.6_1.stl" scale="0.001 0.001 0.001"/>
-    </geometry>
-  </collision>
-</link>
-<link name="wheel_roller1.11_1">
+      <mesh filename="package://deep_ballbot_description/meshes/wheel_roller1_6_1.stl" scale="0.001 0.001 0.001"/>
+    </geometry>
+  </collision>
+</link>
+<link name="wheel_roller1_11_1">
   <inertial>
     <origin rpy="0 0 0" xyz="1.5200671593662562e-07 -6.254028867003214e-08 -3.0009008898657097e-07"/>
@@ -773,5 +773,5 @@
     <origin rpy="0 0 0" xyz="0.037783 -0.051814 -0.113781"/>
     <geometry>
-      <mesh filename="package://deep_ballbot_description/meshes/wheel_roller1.11_1.stl" scale="0.001 0.001 0.001"/>
+      <mesh filename="package://deep_ballbot_description/meshes/wheel_roller1_11_1.stl" scale="0.001 0.001 0.001"/>
     </geometry>
     <material name="silver"/>
@@ -780,9 +780,9 @@
     <origin rpy="0 0 0" xyz="0.037783 -0.051814 -0.113781"/>
     <geometry>
-      <mesh filename="package://deep_ballbot_description/meshes/wheel_roller1.11_1.stl" scale="0.001 0.001 0.001"/>
-    </geometry>
-  </collision>
-</link>
-<link name="wheel_roller1.3_1">
+      <mesh filename="package://deep_ballbot_description/meshes/wheel_roller1_11_1.stl" scale="0.001 0.001 0.001"/>
+    </geometry>
+  </collision>
+</link>
+<link name="wheel_roller1_3_1">
   <inertial>
     <origin rpy="0 0 0" xyz="1.8441451418022003e-07 4.0516786581346054e-07 3.016277917294863e-07"/>
@@ -793,5 +793,5 @@
     <origin rpy="0 0 0" xyz="0.046834 -0.05735 -0.124387"/>
     <geometry>
-      <mesh filename="package://deep_ballbot_description/meshes/wheel_roller1.3_1.stl" scale="0.001 0.001 0.001"/>
+      <mesh filename="package://deep_ballbot_description/meshes/wheel_roller1_3_1.stl" scale="0.001 0.001 0.001"/>
     </geometry>
     <material name="silver"/>
@@ -800,9 +800,9 @@
     <origin rpy="0 0 0" xyz="0.046834 -0.05735 -0.124387"/>
     <geometry>
-      <mesh filename="package://deep_ballbot_description/meshes/wheel_roller1.3_1.stl" scale="0.001 0.001 0.001"/>
-    </geometry>
-  </collision>
-</link>
-<link name="wheel_roller1.8_1">
+      <mesh filename="package://deep_ballbot_description/meshes/wheel_roller1_3_1.stl" scale="0.001 0.001 0.001"/>
+    </geometry>
+  </collision>
+</link>
+<link name="wheel_roller1_8_1">
   <inertial>
     <origin rpy="0 0 0" xyz="-2.1064078460641955e-08 -4.6082251386331263e-07 -9.665432529337714e-08"/>
@@ -813,5 +813,5 @@
     <origin rpy="0 0 0" xyz="0.056154 -0.062421 -0.134994"/>
     <geometry>
-      <mesh filename="package://deep_ballbot_description/meshes/wheel_roller1.8_1.stl" scale="0.001 0.001 0.001"/>
+      <mesh filename="package://deep_ballbot_description/meshes/wheel_roller1_8_1.stl" scale="0.001 0.001 0.001"/>
     </geometry>
     <material name="silver"/>
@@ -820,9 +820,9 @@
     <origin rpy="0 0 0" xyz="0.056154 -0.062421 -0.134994"/>
     <geometry>
-      <mesh filename="package://deep_ballbot_description/meshes/wheel_roller1.8_1.stl" scale="0.001 0.001 0.001"/>
-    </geometry>
-  </collision>
-</link>
-<link name="wheel_roller1.1_1">
+      <mesh filename="package://deep_ballbot_description/meshes/wheel_roller1_8_1.stl" scale="0.001 0.001 0.001"/>
+    </geometry>
+  </collision>
+</link>
+<link name="wheel_roller1_1_1">
   <inertial>
     <origin rpy="0 0 0" xyz="-4.803400587422013e-07 2.0996169430853584e-07 7.806477037020088e-08"/>
@@ -833,5 +833,5 @@
     <origin rpy="0 0 0" xyz="0.067317 -0.054021 -0.140462"/>
     <geometry>
-      <mesh filename="package://deep_ballbot_description/meshes/wheel_roller1.1_1.stl" scale="0.001 0.001 0.001"/>
+      <mesh filename="package://deep_ballbot_description/meshes/wheel_roller1_1_1.stl" scale="0.001 0.001 0.001"/>
     </geometry>
     <material name="silver"/>
@@ -840,9 +840,9 @@
     <origin rpy="0 0 0" xyz="0.067317 -0.054021 -0.140462"/>
     <geometry>
-      <mesh filename="package://deep_ballbot_description/meshes/wheel_roller1.1_1.stl" scale="0.001 0.001 0.001"/>
-    </geometry>
-  </collision>
-</link>
-<link name="wheel_roller2.2_1">
+      <mesh filename="package://deep_ballbot_description/meshes/wheel_roller1_1_1.stl" scale="0.001 0.001 0.001"/>
+    </geometry>
+  </collision>
+</link>
+<link name="wheel_roller2_2_1">
   <inertial>
     <origin rpy="0 0 0" xyz="3.3311915409890104e-17 3.199273256454527e-07 -4.949365299544706e-07"/>
@@ -853,5 +853,5 @@
     <origin rpy="0 0 0" xyz="-0.0 0.090448 -0.145601"/>
     <geometry>
-      <mesh filename="package://deep_ballbot_description/meshes/wheel_roller2.2_1.stl" scale="0.001 0.001 0.001"/>
+      <mesh filename="package://deep_ballbot_description/meshes/wheel_roller2_2_1.stl" scale="0.001 0.001 0.001"/>
     </geometry>
     <material name="silver"/>
@@ -860,9 +860,9 @@
     <origin rpy="0 0 0" xyz="-0.0 0.090448 -0.145601"/>
     <geometry>
-      <mesh filename="package://deep_ballbot_description/meshes/wheel_roller2.2_1.stl" scale="0.001 0.001 0.001"/>
-    </geometry>
-  </collision>
-</link>
-<link name="wheel_roller2.4_1">
+      <mesh filename="package://deep_ballbot_description/meshes/wheel_roller2_2_1.stl" scale="0.001 0.001 0.001"/>
+    </geometry>
+  </collision>
+</link>
+<link name="wheel_roller2_4_1">
   <inertial>
     <origin rpy="0 0 0" xyz="0.0012986987297727726 0.0015200692565425222 -0.0025402442653456037"/>
@@ -873,5 +873,5 @@
     <origin rpy="0 0 0" xyz="-0.011783 0.086847 -0.14302"/>
     <geometry>
-      <mesh filename="package://deep_ballbot_description/meshes/wheel_roller2.4_1.stl" scale="0.001 0.001 0.001"/>
+      <mesh filename="package://deep_ballbot_description/meshes/wheel_roller2_4_1.stl" scale="0.001 0.001 0.001"/>
     </geometry>
     <material name="silver"/>
@@ -880,9 +880,9 @@
     <origin rpy="0 0 0" xyz="-0.011783 0.086847 -0.14302"/>
     <geometry>
-      <mesh filename="package://deep_ballbot_description/meshes/wheel_roller2.4_1.stl" scale="0.001 0.001 0.001"/>
-    </geometry>
-  </collision>
-</link>
-<link name="wheel_roller2.7_1">
+      <mesh filename="package://deep_ballbot_description/meshes/wheel_roller2_4_1.stl" scale="0.001 0.001 0.001"/>
+    </geometry>
+  </collision>
+</link>
+<link name="wheel_roller2_7_1">
   <inertial>
     <origin rpy="0 0 0" xyz="-2.3788655219292298e-07 -7.835488179119832e-08 -9.665444469786344e-08"/>
@@ -893,5 +893,5 @@
     <origin rpy="0 0 0" xyz="-0.025981 0.079841 -0.134994"/>
     <geometry>
-      <mesh filename="package://deep_ballbot_description/meshes/wheel_roller2.7_1.stl" scale="0.001 0.001 0.001"/>
+      <mesh filename="package://deep_ballbot_description/meshes/wheel_roller2_7_1.stl" scale="0.001 0.001 0.001"/>
     </geometry>
     <material name="silver"/>
@@ -900,9 +900,9 @@
     <origin rpy="0 0 0" xyz="-0.025981 0.079841 -0.134994"/>
     <geometry>
-      <mesh filename="package://deep_ballbot_description/meshes/wheel_roller2.7_1.stl" scale="0.001 0.001 0.001"/>
-    </geometry>
-  </collision>
-</link>
-<link name="wheel_roller2.12_1">
+      <mesh filename="package://deep_ballbot_description/meshes/wheel_roller2_7_1.stl" scale="0.001 0.001 0.001"/>
+    </geometry>
+  </collision>
+</link>
+<link name="wheel_roller2_12_1">
   <inertial>
     <origin rpy="0 0 0" xyz="-4.1071313017226885e-14 -4.7663711796874786e-07 3.0162779128539707e-07"/>
@@ -913,5 +913,5 @@
     <origin rpy="0 0 0" xyz="-0.02625 0.069234 -0.124387"/>
     <geometry>
-      <mesh filename="package://deep_ballbot_description/meshes/wheel_roller2.12_1.stl" scale="0.001 0.001 0.001"/>
+      <mesh filename="package://deep_ballbot_description/meshes/wheel_roller2_12_1.stl" scale="0.001 0.001 0.001"/>
     </geometry>
     <material name="silver"/>
@@ -920,9 +920,9 @@
     <origin rpy="0 0 0" xyz="-0.02625 0.069234 -0.124387"/>
     <geometry>
-      <mesh filename="package://deep_ballbot_description/meshes/wheel_roller2.12_1.stl" scale="0.001 0.001 0.001"/>
-    </geometry>
-  </collision>
-</link>
-<link name="wheel_roller2.9_1">
+      <mesh filename="package://deep_ballbot_description/meshes/wheel_roller2_12_1.stl" scale="0.001 0.001 0.001"/>
+    </geometry>
+  </collision>
+</link>
+<link name="wheel_roller2_9_1">
   <inertial>
     <origin rpy="0 0 0" xyz="-2.378865546909248e-07 1.356287089582242e-09 -1.763656140435499e-07"/>
@@ -933,5 +933,5 @@
     <origin rpy="0 0 0" xyz="-0.025986 0.058634 -0.113787"/>
     <geometry>
-      <mesh filename="package://deep_ballbot_description/meshes/wheel_roller2.9_1.stl" scale="0.001 0.001 0.001"/>
+      <mesh filename="package://deep_ballbot_description/meshes/wheel_roller2_9_1.stl" scale="0.001 0.001 0.001"/>
     </geometry>
     <material name="silver"/>
@@ -940,9 +940,9 @@
     <origin rpy="0 0 0" xyz="-0.025986 0.058634 -0.113787"/>
     <geometry>
-      <mesh filename="package://deep_ballbot_description/meshes/wheel_roller2.9_1.stl" scale="0.001 0.001 0.001"/>
-    </geometry>
-  </collision>
-</link>
-<link name="wheel_roller2.5_1">
+      <mesh filename="package://deep_ballbot_description/meshes/wheel_roller2_9_1.stl" scale="0.001 0.001 0.001"/>
+    </geometry>
+  </collision>
+</link>
+<link name="wheel_roller2_5_1">
   <inertial>
     <origin rpy="0 0 0" xyz="-3.3974599707858877e-07 -2.3573421648048765e-07 6.072436552206906e-08"/>
@@ -953,5 +953,5 @@
     <origin rpy="0 0 0" xyz="-0.013134 0.053163 -0.108316"/>
     <geometry>
-      <mesh filename="package://deep_ballbot_description/meshes/wheel_roller2.5_1.stl" scale="0.001 0.001 0.001"/>
+      <mesh filename="package://deep_ballbot_description/meshes/wheel_roller2_5_1.stl" scale="0.001 0.001 0.001"/>
     </geometry>
     <material name="silver"/>
@@ -960,9 +960,9 @@
     <origin rpy="0 0 0" xyz="-0.013134 0.053163 -0.108316"/>
     <geometry>
-      <mesh filename="package://deep_ballbot_description/meshes/wheel_roller2.5_1.stl" scale="0.001 0.001 0.001"/>
-    </geometry>
-  </collision>
-</link>
-<link name="wheel_roller2.10_1">
+      <mesh filename="package://deep_ballbot_description/meshes/wheel_roller2_5_1.stl" scale="0.001 0.001 0.001"/>
+    </geometry>
+  </collision>
+</link>
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