Commit message: fix: recenter baselink in URDF

File: deep_ballbot_description/urdf/deep_ballbot.xacro (robot description, xacro)
@@ -6,5 +6,5 @@
 <link name="base_link">
   <inertial>
-    <origin rpy="0 0 0" xyz="1.044895162337113e-16 -4.0782779191072703e-16 0.2890000000000001"/>
+    <origin rpy="0 0 0" xyz="1.2837111033282416e-16 -5.2625812969710457e-17 0.19100000000000006"/>
     <mass value="0.1429407"/>
     <inertia ixx="0.001077" ixy="-0.0" ixz="0.0" iyy="0.001077" iyz="0.0" izz="1.1e-05"/>
@@ -26,10 +26,10 @@
 <link name="base_shell1_1">
   <inertial>
-    <origin rpy="0 0 0" xyz="-0.03154930294610876 0.01821499854868268 0.021364464404157207"/>
+    <origin rpy="0 0 0" xyz="-0.031549302946108734 0.018214998548683036 0.021364464404157207"/>
     <mass value="0.03897424370875784"/>
     <inertia ixx="3.3e-05" ixy="-1.1e-05" ixz="6e-06" iyy="2e-05" iyz="-3e-06" izz="3.8e-05"/>
   </inertial>
   <visual>
-    <origin rpy="0 0 0" xyz="-0.0 -0.0 -0.139"/>
+    <origin rpy="0 0 0" xyz="-0.0 -0.0 -0.041"/>
     <geometry>
       <mesh filename="package://deep_ballbot_description/meshes/base_shell1_1.stl" scale="0.001 0.001 0.001"/>
@@ -38,5 +38,5 @@
   </visual>
   <collision>
-    <origin rpy="0 0 0" xyz="-0.0 -0.0 -0.139"/>
+    <origin rpy="0 0 0" xyz="-0.0 -0.0 -0.041"/>
     <geometry>
       <mesh filename="package://deep_ballbot_description/meshes/base_shell1_1.stl" scale="0.001 0.001 0.001"/>
@@ -46,10 +46,10 @@
 <link name="base_shell2_1">
   <inertial>
-    <origin rpy="0 0 0" xyz="-3.417367020505995e-15 -0.037022459667432825 0.022039444136548486"/>
+    <origin rpy="0 0 0" xyz="-3.3934854264068832e-15 -0.03702245966743248 0.022039444136548507"/>
     <mass value="0.037632056653399956"/>
     <inertia ixx="1.3e-05" ixy="-0.0" ixz="-0.0" iyy="3.8e-05" iyz="6e-06" izz="3.7e-05"/>
   </inertial>
   <visual>
-    <origin rpy="0 0 0" xyz="-0.0 -0.0 -0.139"/>
+    <origin rpy="0 0 0" xyz="-0.0 -0.0 -0.041"/>
     <geometry>
       <mesh filename="package://deep_ballbot_description/meshes/base_shell2_1.stl" scale="0.001 0.001 0.001"/>
@@ -58,5 +58,5 @@
   </visual>
   <collision>
-    <origin rpy="0 0 0" xyz="-0.0 -0.0 -0.139"/>
+    <origin rpy="0 0 0" xyz="-0.0 -0.0 -0.041"/>
     <geometry>
       <mesh filename="package://deep_ballbot_description/meshes/base_shell2_1.stl" scale="0.001 0.001 0.001"/>
@@ -66,10 +66,10 @@
 <link name="base_shell3_1">
   <inertial>
-    <origin rpy="0 0 0" xyz="0.0315493029461081 0.01821499854867909 0.021364464404157207"/>
+    <origin rpy="0 0 0" xyz="0.031549302946108124 0.01821499854867945 0.021364464404157207"/>
     <mass value="0.03897424370875779"/>
     <inertia ixx="3.3e-05" ixy="1.1e-05" ixz="-6e-06" iyy="2e-05" iyz="-3e-06" izz="3.8e-05"/>
   </inertial>
   <visual>
-    <origin rpy="0 0 0" xyz="-0.0 -0.0 -0.139"/>
+    <origin rpy="0 0 0" xyz="-0.0 -0.0 -0.041"/>
     <geometry>
       <mesh filename="package://deep_ballbot_description/meshes/base_shell3_1.stl" scale="0.001 0.001 0.001"/>
@@ -78,5 +78,5 @@
   </visual>
   <collision>
-    <origin rpy="0 0 0" xyz="-0.0 -0.0 -0.139"/>
+    <origin rpy="0 0 0" xyz="-0.0 -0.0 -0.041"/>
     <geometry>
       <mesh filename="package://deep_ballbot_description/meshes/base_shell3_1.stl" scale="0.001 0.001 0.001"/>
@@ -86,10 +86,10 @@
 <link name="base_plate2_1">
   <inertial>
-    <origin rpy="0 0 0" xyz="-0.008447575075313324 0.0259707939694059 0.0029137797806522425"/>
+    <origin rpy="0 0 0" xyz="-0.008447575075313303 0.025970793969406256 0.0029137797806522286"/>
     <mass value="0.029331775102842923"/>
     <inertia ixx="1.5e-05" ixy="-6e-06" ixz="-0.0" iyy="9e-06" iyz="0.0" izz="2.4e-05"/>
   </inertial>
   <visual>
-    <origin rpy="0 0 0" xyz="-0.040768 0.044631 -0.184"/>
+    <origin rpy="0 0 0" xyz="-0.040768 0.044631 -0.086"/>
     <geometry>
       <mesh filename="package://deep_ballbot_description/meshes/base_plate2_1.stl" scale="0.001 0.001 0.001"/>
@@ -98,5 +98,5 @@
   </visual>
   <collision>
-    <origin rpy="0 0 0" xyz="-0.040768 0.044631 -0.184"/>
+    <origin rpy="0 0 0" xyz="-0.040768 0.044631 -0.086"/>
     <geometry>
       <mesh filename="package://deep_ballbot_description/meshes/base_plate2_1.stl" scale="0.001 0.001 0.001"/>
@@ -106,10 +106,10 @@
 <link name="base_plate3_1">
   <inertial>
-    <origin rpy="0 0 0" xyz="-0.018267999999997092 -0.02030158793881661 0.002913779780652437"/>
+    <origin rpy="0 0 0" xyz="-0.018267999999997068 -0.020301587938816257 0.002913779780652437"/>
     <mass value="0.029331775102842902"/>
     <inertia ixx="5e-06" ixy="-0.0" ixz="0.0" iyy="1.9e-05" iyz="-0.0" izz="2.4e-05"/>
   </inertial>
   <visual>
-    <origin rpy="0 0 0" xyz="-0.018268 -0.057622 -0.184"/>
+    <origin rpy="0 0 0" xyz="-0.018268 -0.057622 -0.086"/>
     <geometry>
       <mesh filename="package://deep_ballbot_description/meshes/base_plate3_1.stl" scale="0.001 0.001 0.001"/>
@@ -118,5 +118,5 @@
   </visual>
   <collision>
-    <origin rpy="0 0 0" xyz="-0.018268 -0.057622 -0.184"/>
+    <origin rpy="0 0 0" xyz="-0.018268 -0.057622 -0.086"/>
     <geometry>
       <mesh filename="package://deep_ballbot_description/meshes/base_plate3_1.stl" scale="0.001 0.001 0.001"/>
@@ -126,10 +126,10 @@
 <link name="vertical_bay1_1">
   <inertial>
-    <origin rpy="0 0 0" xyz="-1.6167557852567183e-07 1.1086679559124679e-07 0.03426796949760952"/>
+    <origin rpy="0 0 0" xyz="-1.616755785013857e-07 1.108667959468651e-07 0.034267969497609505"/>
     <mass value="0.02673500652833671"/>
     <inertia ixx="1.7e-05" ixy="4e-06" ixz="0.0" iyy="1.3e-05" iyz="0.0" izz="8e-06"/>
   </inertial>
   <visual>
-    <origin rpy="0 0 0" xyz="0.023921 0.013811 -0.187"/>
+    <origin rpy="0 0 0" xyz="0.023921 0.013811 -0.089"/>
     <geometry>
       <mesh filename="package://deep_ballbot_description/meshes/vertical_bay1_1.stl" scale="0.001 0.001 0.001"/>
@@ -138,5 +138,5 @@
   </visual>
   <collision>
-    <origin rpy="0 0 0" xyz="0.023921 0.013811 -0.187"/>
+    <origin rpy="0 0 0" xyz="0.023921 0.013811 -0.089"/>
     <geometry>
       <mesh filename="package://deep_ballbot_description/meshes/vertical_bay1_1.stl" scale="0.001 0.001 0.001"/>
@@ -146,10 +146,10 @@
 <link name="vertical_bay2_1">
   <inertial>
-    <origin rpy="0 0 0" xyz="1.6167524612489825e-07 1.108674625403816e-07 0.034307521329889706"/>
+    <origin rpy="0 0 0" xyz="1.6167524614571493e-07 1.1086746289426519e-07 0.034307521329889665"/>
     <mass value="0.026769047843990496"/>
     <inertia ixx="1.8e-05" ixy="-4e-06" ixz="0.0" iyy="1.3e-05" iyz="-0.0" izz="8e-06"/>
   </inertial>
   <visual>
-    <origin rpy="0 0 0" xyz="-0.023921 0.013811 -0.187"/>
+    <origin rpy="0 0 0" xyz="-0.023921 0.013811 -0.089"/>
     <geometry>
       <mesh filename="package://deep_ballbot_description/meshes/vertical_bay2_1.stl" scale="0.001 0.001 0.001"/>
@@ -158,5 +158,5 @@
   </visual>
   <collision>
-    <origin rpy="0 0 0" xyz="-0.023921 0.013811 -0.187"/>
+    <origin rpy="0 0 0" xyz="-0.023921 0.013811 -0.089"/>
     <geometry>
       <mesh filename="package://deep_ballbot_description/meshes/vertical_bay2_1.stl" scale="0.001 0.001 0.001"/>
@@ -166,10 +166,10 @@
 <link name="vertical_bay3_1">
   <inertial>
-    <origin rpy="0 0 0" xyz="4.8585964403268e-15 -2.2173493367805275e-07 0.03430752132988982"/>
+    <origin rpy="0 0 0" xyz="4.882478034425914e-15 -2.217349333276386e-07 0.03430752132988979"/>
     <mass value="0.026769047843990493"/>
     <inertia ixx="1.1e-05" ixy="-0.0" ixz="-0.0" iyy="2e-05" iyz="0.0" izz="8e-06"/>
   </inertial>
   <visual>
-    <origin rpy="0 0 0" xyz="-0.0 -0.027622 -0.187"/>
+    <origin rpy="0 0 0" xyz="-0.0 -0.027622 -0.089"/>
     <geometry>
       <mesh filename="package://deep_ballbot_description/meshes/vertical_bay3_1.stl" scale="0.001 0.001 0.001"/>
@@ -178,5 +178,5 @@
   </visual>
   <collision>
-    <origin rpy="0 0 0" xyz="-0.0 -0.027622 -0.187"/>
+    <origin rpy="0 0 0" xyz="-0.0 -0.027622 -0.089"/>
     <geometry>
       <mesh filename="package://deep_ballbot_description/meshes/vertical_bay3_1.stl" scale="0.001 0.001 0.001"/>
@@ -186,10 +186,10 @@
 <link name="breadboard_1">
   <inertial>
-    <origin rpy="0 0 0" xyz="-3.512780628184276e-10 0.017499602320883354 0.003999999999999948"/>
+    <origin rpy="0 0 0" xyz="-3.5127803936496616e-10 0.017499602320883708 0.00399999999999992"/>
     <mass value="0.016254000000000088"/>
     <inertia ixx="2e-06" ixy="-0.0" ixz="-0.0" iyy="3e-06" iyz="0.0" izz="4e-06"/>
   </inertial>
   <visual>
-    <origin rpy="0 0 0" xyz="0.0 0.047631 -0.258"/>
+    <origin rpy="0 0 0" xyz="0.0 0.047631 -0.16"/>
     <geometry>
       <mesh filename="package://deep_ballbot_description/meshes/breadboard_1.stl" scale="0.001 0.001 0.001"/>
@@ -198,5 +198,5 @@
   </visual>
   <collision>
-    <origin rpy="0 0 0" xyz="0.0 0.047631 -0.258"/>
+    <origin rpy="0 0 0" xyz="0.0 0.047631 -0.16"/>
     <geometry>
       <mesh filename="package://deep_ballbot_description/meshes/breadboard_1.stl" scale="0.001 0.001 0.001"/>
@@ -206,5 +206,5 @@
 <link name="arduino_nano_1">
   <inertial>
-    <origin rpy="0 0 0" xyz="-0.0015922703223249265 0.0015396023112441357 0.014355883406889147"/>
+    <origin rpy="0 0 0" xyz="-0.0015922703223249027 0.001539602311244493 -0.08364411659311086"/>
     <mass value="0.014605507737955568"/>
     <inertia ixx="1e-06" ixy="-0.0" ixz="0.0" iyy="2e-06" iyz="0.0" izz="3e-06"/>
@@ -226,10 +226,10 @@
 <link name="rasbperry_pi_1">
   <inertial>
-    <origin rpy="0 0 0" xyz="-0.0012540090701389588 0.004888830200196736 0.057465472519733274"/>
+    <origin rpy="0 0 0" xyz="-0.0012540090701389367 0.004888830200197092 0.057465472519733246"/>
     <mass value="0.13472167579144456"/>
     <inertia ixx="8.3e-05" ixy="0.0" ixz="-0.0" iyy="0.000118" iyz="-9e-06" izz="4.1e-05"/>
   </inertial>
   <visual>
-    <origin rpy="0 0 0" xyz="0.0 -0.0105 -0.258"/>
+    <origin rpy="0 0 0" xyz="0.0 -0.0105 -0.16"/>
     <geometry>
       <mesh filename="package://deep_ballbot_description/meshes/rasbperry_pi_1.stl" scale="0.001 0.001 0.001"/>
@@ -238,5 +238,5 @@
   </visual>
   <collision>
-    <origin rpy="0 0 0" xyz="0.0 -0.0105 -0.258"/>
+    <origin rpy="0 0 0" xyz="0.0 -0.0105 -0.16"/>
     <geometry>
       <mesh filename="package://deep_ballbot_description/meshes/rasbperry_pi_1.stl" scale="0.001 0.001 0.001"/>
@@ -246,10 +246,10 @@
 <link name="motor_mount1_1">
   <inertial>
-    <origin rpy="0 0 0" xyz="0.008784093083896216 -0.005071216542772684 -0.01575982915390231"/>
+    <origin rpy="0 0 0" xyz="0.008784093083896244 -0.005071216542772327 -0.01575982915390229"/>
     <mass value="0.08608420182582005"/>
     <inertia ixx="3.8e-05" ixy="-9e-06" ixz="1e-05" iyy="2.8e-05" iyz="-6e-06" izz="4.3e-05"/>
   </inertial>
   <visual>
-    <origin rpy="0 0 0" xyz="0.046487 -0.026839 -0.171056"/>
+    <origin rpy="0 0 0" xyz="0.046487 -0.026839 -0.073056"/>
     <geometry>
       <mesh filename="package://deep_ballbot_description/meshes/motor_mount1_1.stl" scale="0.001 0.001 0.001"/>
@@ -258,5 +258,5 @@
   </visual>
   <collision>
-    <origin rpy="0 0 0" xyz="0.046487 -0.026839 -0.171056"/>
+    <origin rpy="0 0 0" xyz="0.046487 -0.026839 -0.073056"/>
     <geometry>
       <mesh filename="package://deep_ballbot_description/meshes/motor_mount1_1.stl" scale="0.001 0.001 0.001"/>
@@ -266,10 +266,10 @@
 <link name="motor_mount2_1">
   <inertial>
-    <origin rpy="0 0 0" xyz="1.2758713609389452e-14 0.010142433085668257 -0.01575982915375221"/>
+    <origin rpy="0 0 0" xyz="1.2782595203488562e-14 0.01014243308566861 -0.015759829153752188"/>
     <mass value="0.08608420182581958"/>
     <inertia ixx="2.3e-05" ixy="0.0" ixz="-0.0" iyy="4.3e-05" iyz="1.1e-05" izz="4.3e-05"/>
   </inertial>
   <visual>
-    <origin rpy="0 0 0" xyz="-0.0 0.053678 -0.171056"/>
+    <origin rpy="0 0 0" xyz="-0.0 0.053678 -0.073056"/>
     <geometry>
       <mesh filename="package://deep_ballbot_description/meshes/motor_mount2_1.stl" scale="0.001 0.001 0.001"/>
@@ -278,5 +278,5 @@
   </visual>
   <collision>
-    <origin rpy="0 0 0" xyz="-0.0 0.053678 -0.171056"/>
+    <origin rpy="0 0 0" xyz="-0.0 0.053678 -0.073056"/>
     <geometry>
       <mesh filename="package://deep_ballbot_description/meshes/motor_mount2_1.stl" scale="0.001 0.001 0.001"/>
@@ -286,10 +286,10 @@
 <link name="motor_mount3_1">
   <inertial>
-    <origin rpy="0 0 0" xyz="-0.008784093083910476 -0.005071216542747357 -0.015759829153902005"/>
+    <origin rpy="0 0 0" xyz="-0.008784093083910455 -0.0050712165427470035 -0.015759829153901964"/>
     <mass value="0.08608420182581962"/>
     <inertia ixx="3.8e-05" ixy="9e-06" ixz="-1e-05" iyy="2.8e-05" iyz="-6e-06" izz="4.3e-05"/>
   </inertial>
   <visual>
-    <origin rpy="0 0 0" xyz="-0.046487 -0.026839 -0.171056"/>
+    <origin rpy="0 0 0" xyz="-0.046487 -0.026839 -0.073056"/>
     <geometry>
       <mesh filename="package://deep_ballbot_description/meshes/motor_mount3_1.stl" scale="0.001 0.001 0.001"/>
@@ -298,5 +298,5 @@
   </visual>
   <collision>
-    <origin rpy="0 0 0" xyz="-0.046487 -0.026839 -0.171056"/>
+    <origin rpy="0 0 0" xyz="-0.046487 -0.026839 -0.073056"/>
     <geometry>
       <mesh filename="package://deep_ballbot_description/meshes/motor_mount3_1.stl" scale="0.001 0.001 0.001"/>
@@ -306,10 +306,10 @@
 <link name="arduino_mount1_1">
   <inertial>
-    <origin rpy="0 0 0" xyz="-0.0017985403607222034 -0.0017781689855505562 -2.1615661864288205e-05"/>
+    <origin rpy="0 0 0" xyz="-0.0017985403607221756 -0.0017781689855501989 -2.161566186426045e-05"/>
     <mass value="0.023201510107992093"/>
     <inertia ixx="1.3e-05" ixy="5e-06" ixz="-0.0" iyy="8e-06" iyz="0.0" izz="1.2e-05"/>
   </inertial>
   <visual>
-    <origin rpy="0 0 0" xyz="0.026519 0.015311 -0.2195"/>
+    <origin rpy="0 0 0" xyz="0.026519 0.015311 -0.1215"/>
     <geometry>
       <mesh filename="package://deep_ballbot_description/meshes/arduino_mount1_1.stl" scale="0.001 0.001 0.001"/>
@@ -318,5 +318,5 @@
   </visual>
   <collision>
-    <origin rpy="0 0 0" xyz="0.026519 0.015311 -0.2195"/>
+    <origin rpy="0 0 0" xyz="0.026519 0.015311 -0.1215"/>
     <geometry>
       <mesh filename="package://deep_ballbot_description/meshes/arduino_mount1_1.stl" scale="0.001 0.001 0.001"/>
@@ -326,10 +326,10 @@
 <link name="arduino_mount2_1">
   <inertial>
-    <origin rpy="0 0 0" xyz="0.0024394246518729297 -0.0006681248315038978 -2.1615661864288205e-05"/>
+    <origin rpy="0 0 0" xyz="0.002439424651872954 -0.0006681248315035439 -2.1615661864302083e-05"/>
     <mass value="0.023201510107960607"/>
     <inertia ixx="1.3e-05" ixy="-5e-06" ixz="-0.0" iyy="8e-06" iyz="-0.0" izz="1.2e-05"/>
   </inertial>
   <visual>
-    <origin rpy="0 0 0" xyz="-0.026519 0.015311 -0.2195"/>
+    <origin rpy="0 0 0" xyz="-0.026519 0.015311 -0.1215"/>
     <geometry>
       <mesh filename="package://deep_ballbot_description/meshes/arduino_mount2_1.stl" scale="0.001 0.001 0.001"/>
@@ -338,5 +338,5 @@
   </visual>
   <collision>
-    <origin rpy="0 0 0" xyz="-0.026519 0.015311 -0.2195"/>
+    <origin rpy="0 0 0" xyz="-0.026519 0.015311 -0.1215"/>
     <geometry>
       <mesh filename="package://deep_ballbot_description/meshes/arduino_mount2_1.stl" scale="0.001 0.001 0.001"/>
@@ -346,10 +346,10 @@
 <link name="arduino_mount3_1">
   <inertial>
-    <origin rpy="0 0 0" xyz="-0.0006408842911585192 0.0024462938179583525 -2.1615661864482494e-05"/>
+    <origin rpy="0 0 0" xyz="-0.0006408842911584954 0.0024462938179587064 -2.161566186449637e-05"/>
     <mass value="0.023201510107976293"/>
     <inertia ixx="5e-06" ixy="0.0" ixz="0.0" iyy="1.6e-05" iyz="0.0" izz="1.2e-05"/>
   </inertial>
   <visual>
-    <origin rpy="0 0 0" xyz="-0.0 -0.030622 -0.2195"/>
+    <origin rpy="0 0 0" xyz="-0.0 -0.030622 -0.1215"/>
     <geometry>
       <mesh filename="package://deep_ballbot_description/meshes/arduino_mount3_1.stl" scale="0.001 0.001 0.001"/>
@@ -358,5 +358,5 @@
   </visual>
   <collision>
-    <origin rpy="0 0 0" xyz="-0.0 -0.030622 -0.2195"/>
+    <origin rpy="0 0 0" xyz="-0.0 -0.030622 -0.1215"/>
     <geometry>
       <mesh filename="package://deep_ballbot_description/meshes/arduino_mount3_1.stl" scale="0.001 0.001 0.001"/>
@@ -366,10 +366,10 @@
 <link name="arduino1_1">
   <inertial>
-    <origin rpy="0 0 0" xyz="0.01666958536509317 -0.034661355386450377 0.00875853373784699"/>
+    <origin rpy="0 0 0" xyz="0.016669585365093192 -0.03466135538645002 0.008758533737846977"/>
     <mass value="0.0763619336554754"/>
     <inertia ixx="4.9e-05" ixy="1.4e-05" ixz="0.0" iyy="2.9e-05" iyz="-1e-06" izz="3.5e-05"/>
   </inertial>
   <visual>
-    <origin rpy="0 0 0" xyz="0.047078 -0.010299 -0.211"/>
+    <origin rpy="0 0 0" xyz="0.047078 -0.010299 -0.113"/>
     <geometry>
       <mesh filename="package://deep_ballbot_description/meshes/arduino1_1.stl" scale="0.001 0.001 0.001"/>
@@ -378,5 +378,5 @@
   </visual>
   <collision>
-    <origin rpy="0 0 0" xyz="0.047078 -0.010299 -0.211"/>
+    <origin rpy="0 0 0" xyz="0.047078 -0.010299 -0.113"/>
     <geometry>
       <mesh filename="package://deep_ballbot_description/meshes/arduino1_1.stl" scale="0.001 0.001 0.001"/>
@@ -386,10 +386,10 @@
 <link name="arduino2_1">
   <inertial>
-    <origin rpy="0 0 0" xyz="0.021682625979238306 0.03176671812995284 0.008758533737850571"/>
+    <origin rpy="0 0 0" xyz="0.021682625979238333 0.0317667181299532 0.008758533737850557"/>
     <mass value="0.07636193365547596"/>
     <inertia ixx="4.6e-05" ixy="-1.6e-05" ixz="1e-06" iyy="3.2e-05" iyz="1e-06" izz="3.5e-05"/>
   </inertial>
   <visual>
-    <origin rpy="0 0 0" xyz="-0.01462 0.04592 -0.211"/>
+    <origin rpy="0 0 0" xyz="-0.01462 0.04592 -0.113"/>
     <geometry>
       <mesh filename="package://deep_ballbot_description/meshes/arduino2_1.stl" scale="0.001 0.001 0.001"/>
@@ -398,5 +398,5 @@
   </visual>
   <collision>
-    <origin rpy="0 0 0" xyz="-0.01462 0.04592 -0.211"/>
+    <origin rpy="0 0 0" xyz="-0.01462 0.04592 -0.113"/>
     <geometry>
       <mesh filename="package://deep_ballbot_description/meshes/arduino2_1.stl" scale="0.001 0.001 0.001"/>
@@ -406,10 +406,10 @@
 <link name="arduino3_1">
   <inertial>
-    <origin rpy="0 0 0" xyz="-0.03835221134344281 0.0028936372564971197 0.008758533737798002"/>
+    <origin rpy="0 0 0" xyz="-0.03835221134344279 0.0028936372564974805 0.008758533737797974"/>
     <mass value="0.07636193365547513"/>
     <inertia ixx="2.2e-05" ixy="2e-06" ixz="-1e-06" iyy="5.6e-05" iyz="0.0" izz="3.5e-05"/>
   </inertial>
   <visual>
-    <origin rpy="0 0 0" xyz="-0.032458 -0.035622 -0.211"/>
+    <origin rpy="0 0 0" xyz="-0.032458 -0.035622 -0.113"/>
     <geometry>
       <mesh filename="package://deep_ballbot_description/meshes/arduino3_1.stl" scale="0.001 0.001 0.001"/>
@@ -418,5 +418,5 @@
   </visual>
   <collision>
-    <origin rpy="0 0 0" xyz="-0.032458 -0.035622 -0.211"/>
+    <origin rpy="0 0 0" xyz="-0.032458 -0.035622 -0.113"/>
     <geometry>
       <mesh filename="package://deep_ballbot_description/meshes/arduino3_1.stl" scale="0.001 0.001 0.001"/>
@@ -426,10 +426,10 @@
 <link name="motor_stator1_1">
   <inertial>
-    <origin rpy="0 0 0" xyz="0.013066369938678046 -0.007543151268848507 -0.016105881234575237"/>
+    <origin rpy="0 0 0" xyz="0.013066369938678067 -0.00754315126884815 -0.016105881234575264"/>
     <mass value="0.2071891794839974"/>
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