Commit message: fix: add wheel roller inertias

File: deep_ballbot_description/urdf/deep_ballbot_old.xacro (robot description, xacro)
@@ -8,5 +8,5 @@
     <origin rpy="0 0 0" xyz="7.650202289024707e-17 7.328088508434192e-16 0.19082500000000008"/>
     <mass value="0.14294070000000003"/>
-    <inertia ixx="0.00107748" ixy="0.0" ixz="0.0" iyy="0.00107748" iyz="-0.0" izz="1.086e-05"/>
+    <inertia ixx="0.001077" ixy="0.0" ixz="0.0" iyy="0.001077" iyz="-0.0" izz="1.1e-05"/>
   </inertial>
   <visual>
@@ -28,5 +28,5 @@
     <origin rpy="0 0 0" xyz="-0.03154930294610876 0.018214998548683293 0.021364464404157145"/>
     <mass value="0.03897424370875782"/>
-    <inertia ixx="3.265e-05" ixy="-1.056e-05" ixz="5.6e-06" iyy="2.046e-05" iyz="-3.23e-06" izz="3.779e-05"/>
+    <inertia ixx="3.3e-05" ixy="-1.1e-05" ixz="6e-06" iyy="2e-05" iyz="-3e-06" izz="3.8e-05"/>
   </inertial>
   <visual>
@@ -48,5 +48,5 @@
     <origin rpy="0 0 0" xyz="-3.4440123730969962e-15 -0.03702245966743223 0.022039444136548625"/>
     <mass value="0.037632056653399984"/>
-    <inertia ixx="1.346e-05" ixy="-0.0" ixz="-0.0" iyy="3.819e-05" iyz="6.02e-06" izz="3.735e-05"/>
+    <inertia ixx="1.3e-05" ixy="-0.0" ixz="-0.0" iyy="3.8e-05" iyz="6e-06" izz="3.7e-05"/>
   </inertial>
   <visual>
@@ -68,5 +68,5 @@
     <origin rpy="0 0 0" xyz="0.03154930294610811 0.01821499854867976 0.021364464404157152"/>
     <mass value="0.03897424370875781"/>
-    <inertia ixx="3.265e-05" ixy="1.056e-05" ixz="-5.6e-06" iyy="2.046e-05" iyz="-3.23e-06" izz="3.779e-05"/>
+    <inertia ixx="3.3e-05" ixy="1.1e-05" ixz="-6e-06" iyy="2e-05" iyz="-3e-06" izz="3.8e-05"/>
   </inertial>
   <visual>
@@ -88,5 +88,5 @@
     <origin rpy="0 0 0" xyz="-0.008447575075313345 0.025970793969406637 0.0029137797806522564"/>
     <mass value="0.02933177510284292"/>
-    <inertia ixx="1.538e-05" ixy="-5.87e-06" ixz="-2e-08" iyy="8.6e-06" iyz="1e-08" izz="2.38e-05"/>
+    <inertia ixx="1.5e-05" ixy="-6e-06" ixz="-0.0" iyy="9e-06" iyz="0.0" izz="2.4e-05"/>
   </inertial>
   <visual>
@@ -108,5 +108,5 @@
     <origin rpy="0 0 0" xyz="-0.018267999999997113 -0.02030158793881589 0.0029137797806522703"/>
     <mass value="0.029331775102842895"/>
-    <inertia ixx="5.21e-06" ixy="-0.0" ixz="0.0" iyy="1.876e-05" iyz="-2e-08" izz="2.38e-05"/>
+    <inertia ixx="5e-06" ixy="-0.0" ixz="0.0" iyy="1.9e-05" iyz="-0.0" izz="2.4e-05"/>
   </inertial>
   <visual>
@@ -128,5 +128,5 @@
     <origin rpy="0 0 0" xyz="-1.616755785464885e-07 1.1086679645340436e-07 0.034267969497609505"/>
     <mass value="0.026735006528336703"/>
-    <inertia ixx="1.748e-05" ixy="3.56e-06" ixz="0.0" iyy="1.337e-05" iyz="0.0" izz="8.38e-06"/>
+    <inertia ixx="1.7e-05" ixy="4e-06" ixz="0.0" iyy="1.3e-05" iyz="0.0" izz="8e-06"/>
   </inertial>
   <visual>
@@ -148,5 +148,5 @@
     <origin rpy="0 0 0" xyz="1.6167524609367323e-07 1.1086746340080444e-07 0.03430752132988969"/>
     <mass value="0.026769047843990486"/>
-    <inertia ixx="1.751e-05" ixy="-3.56e-06" ixz="0.0" iyy="1.34e-05" iyz="-0.0" izz="8.38e-06"/>
+    <inertia ixx="1.8e-05" ixy="-4e-06" ixz="0.0" iyy="1.3e-05" iyz="-0.0" izz="8e-06"/>
   </inertial>
   <visual>
@@ -168,5 +168,5 @@
     <origin rpy="0 0 0" xyz="4.811851328225059e-15 -2.2173493282803824e-07 0.03430752132988969"/>
     <mass value="0.026769047843990517"/>
-    <inertia ixx="1.135e-05" ixy="-0.0" ixz="-0.0" iyy="1.957e-05" iyz="0.0" izz="8.38e-06"/>
+    <inertia ixx="1.1e-05" ixy="-0.0" ixz="-0.0" iyy="2e-05" iyz="0.0" izz="8e-06"/>
   </inertial>
   <visual>
@@ -188,5 +188,5 @@
     <origin rpy="0 0 0" xyz="-3.512780858557447e-10 0.017499602320884315 0.004000000000000087"/>
     <mass value="0.016254000000000234"/>
-    <inertia ixx="1.75e-06" ixy="-0.0" ixz="0.0" iyy="2.83e-06" iyz="0.0" izz="4.4e-06"/>
+    <inertia ixx="2e-06" ixy="-0.0" ixz="0.0" iyy="3e-06" iyz="0.0" izz="4e-06"/>
   </inertial>
   <visual>
@@ -208,5 +208,5 @@
     <origin rpy="0 0 0" xyz="-0.0012540090701389846 0.004888830200197087 0.057465472519733274"/>
     <mass value="0.1347216757914446"/>
-    <inertia ixx="8.335e-05" ixy="8e-08" ixz="-2e-08" iyy="0.0001181" iyz="-8.51e-06" izz="4.089e-05"/>
+    <inertia ixx="8.3e-05" ixy="0.0" ixz="-0.0" iyy="0.000118" iyz="-9e-06" izz="4.1e-05"/>
   </inertial>
   <visual>
@@ -226,7 +226,7 @@
 <link name="motor_mount1_1">
   <inertial>
-    <origin rpy="0 0 0" xyz="0.008784093083896063 -0.005071216542772112 -0.015759829153902227"/>
-    <mass value="0.08608420182581994"/>
-    <inertia ixx="3.82e-05" ixy="-8.54e-06" ixz="9.75e-06" iyy="2.835e-05" iyz="-5.63e-06" izz="4.313e-05"/>
+    <origin rpy="0 0 0" xyz="0.008784093083896126 -0.005071216542772053 -0.015759829153902304"/>
+    <mass value="0.08608420182582004"/>
+    <inertia ixx="3.8e-05" ixy="-9e-06" ixz="1e-05" iyy="2.8e-05" iyz="-6e-06" izz="4.3e-05"/>
   </inertial>
   <visual>
@@ -248,5 +248,5 @@
     <origin rpy="0 0 0" xyz="1.275150652894624e-14 0.010142433085668805 -0.015759829153751945"/>
     <mass value="0.08608420182581951"/>
-    <inertia ixx="2.342e-05" ixy="0.0" ixz="-0.0" iyy="4.313e-05" iyz="1.126e-05" izz="4.313e-05"/>
+    <inertia ixx="2.3e-05" ixy="0.0" ixz="-0.0" iyy="4.3e-05" iyz="1.1e-05" izz="4.3e-05"/>
   </inertial>
   <visual>
@@ -268,5 +268,5 @@
     <origin rpy="0 0 0" xyz="-0.00878409308391042 -0.005071216542746816 -0.015759829153902033"/>
     <mass value="0.08608420182581976"/>
-    <inertia ixx="3.82e-05" ixy="8.54e-06" ixz="-9.75e-06" iyy="2.835e-05" iyz="-5.63e-06" izz="4.313e-05"/>
+    <inertia ixx="3.8e-05" ixy="9e-06" ixz="-1e-05" iyy="2.8e-05" iyz="-6e-06" izz="4.3e-05"/>
   </inertial>
   <visual>
@@ -288,5 +288,5 @@
     <origin rpy="0 0 0" xyz="-0.001798540360722238 -0.0017781689855501954 -2.1615661864343716e-05"/>
     <mass value="0.023201510107992145"/>
-    <inertia ixx="1.338e-05" ixy="4.98e-06" ixz="-1e-08" iyy="7.62e-06" iyz="1e-08" izz="1.165e-05"/>
+    <inertia ixx="1.3e-05" ixy="5e-06" ixz="-0.0" iyy="8e-06" iyz="0.0" izz="1.2e-05"/>
   </inertial>
   <visual>
@@ -308,5 +308,5 @@
     <origin rpy="0 0 0" xyz="0.002439424651872895 -0.0006681248315035682 -2.1615661864288205e-05"/>
     <mass value="0.023201510107960607"/>
-    <inertia ixx="1.338e-05" ixy="-4.98e-06" ixz="-1e-08" iyy="7.62e-06" iyz="-1e-08" izz="1.165e-05"/>
+    <inertia ixx="1.3e-05" ixy="-5e-06" ixz="-0.0" iyy="8e-06" iyz="-0.0" izz="1.2e-05"/>
   </inertial>
   <visual>
@@ -328,5 +328,5 @@
     <origin rpy="0 0 0" xyz="-0.0006408842911585431 0.0024462938179587064 -2.1615661864468616e-05"/>
     <mass value="0.023201510107976282"/>
-    <inertia ixx="4.74e-06" ixy="0.0" ixz="2e-08" iyy="1.625e-05" iyz="0.0" izz="1.165e-05"/>
+    <inertia ixx="5e-06" ixy="0.0" ixz="0.0" iyy="1.6e-05" iyz="0.0" izz="1.2e-05"/>
   </inertial>
   <visual>
@@ -348,5 +348,5 @@
     <origin rpy="0 0 0" xyz="0.016669585365093106 -0.03466135538644938 0.008758533737846824"/>
     <mass value="0.0763619336554756"/>
-    <inertia ixx="4.901e-05" ixy="1.38e-05" ixz="3.6e-07" iyy="2.915e-05" iyz="-1.24e-06" izz="3.535e-05"/>
+    <inertia ixx="4.9e-05" ixy="1.4e-05" ixz="0.0" iyy="2.9e-05" iyz="-1e-06" izz="3.5e-05"/>
   </inertial>
   <visual>
@@ -368,5 +368,5 @@
     <origin rpy="0 0 0" xyz="0.02168262597923832 0.031766718129953825 0.008758533737850696"/>
     <mass value="0.07636193365547614"/>
-    <inertia ixx="4.607e-05" ixy="-1.55e-05" ixz="8.9e-07" iyy="3.209e-05" iyz="9.3e-07" izz="3.535e-05"/>
+    <inertia ixx="4.6e-05" ixy="-1.6e-05" ixz="1e-06" iyy="3.2e-05" iyz="1e-06" izz="3.5e-05"/>
   </inertial>
   <visual>
@@ -388,5 +388,5 @@
     <origin rpy="0 0 0" xyz="-0.03835221134345001 0.0028936372564978483 0.008758533737797336"/>
     <mass value="0.07636193365547543"/>
-    <inertia ixx="2.216e-05" ixy="1.7e-06" ixz="-1.25e-06" iyy="5.6e-05" iyz="3.1e-07" izz="3.535e-05"/>
+    <inertia ixx="2.2e-05" ixy="2e-06" ixz="-1e-06" iyy="5.6e-05" iyz="0.0" izz="3.5e-05"/>
   </inertial>
   <visual>
@@ -408,5 +408,5 @@
     <origin rpy="0 0 0" xyz="0.013066369938677859 -0.007543151268847602 -0.01610588123457557"/>
     <mass value="0.2071891794839975"/>
-    <inertia ixx="5.6e-05" ixy="-7.8e-06" ixz="1.579e-05" iyy="4.699e-05" iyz="-9.12e-06" izz="6.052e-05"/>
+    <inertia ixx="5.6e-05" ixy="-8e-06" ixz="1.6e-05" iyy="4.7e-05" iyz="-9e-06" izz="6.1e-05"/>
   </inertial>
   <visual>
@@ -428,5 +428,5 @@
     <origin rpy="0 0 0" xyz="2.153687944363946e-17 0.015087302537697599 -0.01610588123457512"/>
     <mass value="0.20718917948399732"/>
-    <inertia ixx="4.249e-05" ixy="0.0" ixz="-0.0" iyy="6.05e-05" iyz="1.824e-05" izz="6.052e-05"/>
+    <inertia ixx="4.2e-05" ixy="0.0" ixz="-0.0" iyy="6.1e-05" iyz="1.8e-05" izz="6.1e-05"/>
   </inertial>
   <visual>
@@ -448,5 +448,5 @@
     <origin rpy="0 0 0" xyz="-0.013066369938677644 -0.007543151268847845 -0.016105881234575542"/>
     <mass value="0.20718917948399762"/>
-    <inertia ixx="5.6e-05" ixy="7.8e-06" ixz="-1.579e-05" iyy="4.699e-05" iyz="-9.12e-06" izz="6.052e-05"/>
+    <inertia ixx="5.6e-05" ixy="8e-06" ixz="-1.6e-05" iyy="4.7e-05" iyz="-9e-06" izz="6.1e-05"/>
   </inertial>
   <visual>
@@ -468,5 +468,5 @@
     <origin rpy="0 0 0" xyz="-0.005759360727442396 0.0033250114622924744 -0.0066512446583098656"/>
     <mass value="0.3781828720603627"/>
-    <inertia ixx="0.00013618" ixy="-1.852e-05" ixz="3.716e-05" iyy="0.0001148" iyz="-2.146e-05" izz="0.00014687"/>
+    <inertia ixx="0.000136" ixy="-1.9e-05" ixz="3.7e-05" iyy="0.000115" iyz="-2.1e-05" izz="0.000147"/>
   </inertial>
   <visual>
@@ -488,5 +488,5 @@
     <origin rpy="0 0 0" xyz="-7.656656279926752e-13 -0.006651022923255909 -0.0066512446583099"/>
     <mass value="0.3781828720603624"/>
-    <inertia ixx="0.00010411" ixy="-0.0" ixz="-0.0" iyy="0.00014687" iyz="4.291e-05" izz="0.00014687"/>
+    <inertia ixx="0.000104" ixy="-0.0" ixz="-0.0" iyy="0.000147" iyz="4.3e-05" izz="0.000147"/>
   </inertial>
   <visual>
@@ -508,5 +508,5 @@
     <origin rpy="0 0 0" xyz="0.005759360728208256 0.0033250114609660285 -0.006651244658309859"/>
     <mass value="0.37818287206036283"/>
-    <inertia ixx="0.00013618" ixy="1.852e-05" ixz="-3.716e-05" iyy="0.0001148" iyz="-2.146e-05" izz="0.00014687"/>
+    <inertia ixx="0.000136" ixy="1.9e-05" ixz="-3.7e-05" iyy="0.000115" iyz="-2.1e-05" izz="0.000147"/>
   </inertial>
   <visual>
@@ -526,7 +526,7 @@
 <link name="wheel_body1_1">
   <inertial>
-    <origin rpy="0 0 0" xyz="-0.007230828099754484 0.004197926495771144 -0.008396531536062641"/>
-    <mass value="0.017118662469058868"/>
-    <inertia ixx="4.34e-06" ixy="-6.5e-07" ixz="1.3e-06" iyy="3.59e-06" iyz="-7.5e-07" izz="4.72e-06"/>
+    <origin rpy="0 0 0" xyz="-0.007230828099754477 0.004197926495771144 -0.008396531536062644"/>
+    <mass value="0.01711866246905887"/>
+    <inertia ixx="4e-06" ixy="-1e-06" ixz="1e-06" iyy="4e-06" iyz="-1e-06" izz="5e-06"/>
   </inertial>
   <visual>
@@ -546,7 +546,7 @@
 <link name="wheel_body2_1">
   <inertial>
-    <origin rpy="0 0 0" xyz="-2.061845722703404e-05 -0.008361140710824139 -0.008396531491025861"/>
-    <mass value="0.01711866259314621"/>
-    <inertia ixx="3.21e-06" ixy="-0.0" ixz="0.0" iyy="4.72e-06" iyz="1.51e-06" izz="4.72e-06"/>
+    <origin rpy="0 0 0" xyz="-2.0618457227039384e-05 -0.00836114071082407 -0.008396531491025875"/>
+    <mass value="0.017118662593146216"/>
+    <inertia ixx="3e-06" ixy="-0.0" ixz="0.0" iyy="5e-06" iyz="2e-06" izz="5e-06"/>
   </inertial>
   <visual>
@@ -566,7 +566,7 @@
 <link name="wheel_body3_1">
   <inertial>
-    <origin rpy="0 0 0" xyz="0.007251872798830904 0.00416228337410076 -0.008396049445361438"/>
-    <mass value="0.017119124264976974"/>
-    <inertia ixx="4.34e-06" ixy="6.5e-07" ixz="-1.3e-06" iyy="3.59e-06" iyz="-7.5e-07" izz="4.72e-06"/>
+    <origin rpy="0 0 0" xyz="0.007251872798830904 0.00416228337410076 -0.008396049445361434"/>
+    <mass value="0.017119124264976967"/>
+    <inertia ixx="4e-06" ixy="1e-06" ixz="-1e-06" iyy="4e-06" iyz="-1e-06" izz="5e-06"/>
   </inertial>
   <visual>
@@ -588,5 +588,5 @@
     <origin rpy="0 0 0" xyz="1.1343589567669454e-08 -1.5996360053227576e-07 -4.949366530018762e-07"/>
     <mass value="0.0012011377071081653"/>
-    <inertia ixx="3e-08" ixy="-1e-08" ixz="-0.0" iyy="2e-08" iyz="-0.0" izz="3e-08"/>
+    <inertia ixx="0.0" ixy="-0.0" ixz="-0.0" iyy="0.0" iyz="-0.0" izz="0.0"/>
   </inertial>
   <visual>
@@ -608,5 +608,5 @@
     <origin rpy="0 0 0" xyz="-0.0001901390157527244 -0.0013906180530564166 -0.0005302442651772127"/>
     <mass value="0.0025623256301060215"/>
-    <inertia ixx="9e-08" ixy="0.0" ixz="0.0" iyy="1.2e-07" iyz="1e-08" izz="9e-08"/>
+    <inertia ixx="0.0" ixy="0.0" ixz="0.0" iyy="0.0" iyz="0.0" izz="0.0"/>
   </inertial>
   <visual>
@@ -628,5 +628,5 @@
     <origin rpy="0 0 0" xyz="2.168223533494107e-07 -4.6082259186688845e-07 -9.665432621625003e-08"/>
     <mass value="0.0012011377071081348"/>
-    <inertia ixx="3e-08" ixy="0.0" ixz="0.0" iyy="2e-08" iyz="-1e-08" izz="3e-08"/>
+    <inertia ixx="0.0" ixy="0.0" ixz="0.0" iyy="0.0" iyz="-0.0" izz="0.0"/>
   </inertial>
   <visual>
@@ -647,6 +647,6 @@
   <inertial>
     <origin rpy="0 0 0" xyz="1.844145551960219e-07 7.146925419185268e-08 3.016277917294863e-07"/>
-    <mass value="0.0025623256301059876"/>
-    <inertia ixx="1e-07" ixy="-1e-08" ixz="-1e-08" iyy="9e-08" iyz="1e-08" izz="1e-07"/>
+    <mass value="0.0025623256301059855"/>
+    <inertia ixx="0.0" ixy="-0.0" ixz="-0.0" iyy="0.0" iyz="0.0" izz="0.0"/>
   </inertial>
   <visual>
@@ -668,5 +668,5 @@
     <origin rpy="0 0 0" xyz="-4.1340771209097404e-07 -3.308052069104714e-07 -1.763657350890846e-07"/>
     <mass value="0.0012011377071081519"/>
-    <inertia ixx="2e-08" ixy="-0.0" ixz="1e-08" iyy="3e-08" iyz="0.0" izz="3e-08"/>
+    <inertia ixx="0.0" ixy="-0.0" ixz="0.0" iyy="0.0" iyz="0.0" izz="0.0"/>
   </inertial>
   <visual>
@@ -688,5 +688,5 @@
     <origin rpy="0 0 0" xyz="4.57179928789464e-07 -4.6555762324602956e-07 6.072472028342824e-08"/>
     <mass value="0.002562325630106018"/>
-    <inertia ixx="1.1e-07" ixy="1e-08" ixz="-1e-08" iyy="1e-07" iyz="-1e-08" izz="9e-08"/>
+    <inertia ixx="0.0" ixy="0.0" ixz="-0.0" iyy="0.0" iyz="-0.0" izz="0.0"/>
   </inertial>
   <visual>
@@ -708,5 +708,5 @@
     <origin rpy="0 0 0" xyz="3.574854795657112e-07 -3.633992790331997e-07 9.819223634015273e-08"/>
     <mass value="0.0012011377071081634"/>
-    <inertia ixx="3e-08" ixy="-1e-08" ixz="0.0" iyy="2e-08" iyz="0.0" izz="3e-08"/>
+    <inertia ixx="0.0" ixy="-0.0" ixz="0.0" iyy="0.0" iyz="0.0" izz="0.0"/>
   </inertial>
   <visual>
@@ -728,5 +728,5 @@
     <origin rpy="0 0 0" xyz="-1.5083097658352695e-07 4.3352494352721926e-07 -4.748097093606324e-07"/>
     <mass value="0.0025623256301060093"/>
-    <inertia ixx="9e-08" ixy="0.0" ixz="0.0" iyy="1.2e-07" iyz="1e-08" izz="9e-08"/>
+    <inertia ixx="0.0" ixy="0.0" ixz="0.0" iyy="0.0" iyz="0.0" izz="0.0"/>
   </inertial>
   <visual>
@@ -748,5 +748,5 @@
     <origin rpy="0 0 0" xyz="1.5200671603377014e-07 -6.25402882536985e-08 -3.000900884626845e-07"/>
     <mass value="0.0012011377071081484"/>
-    <inertia ixx="3e-08" ixy="0.0" ixz="0.0" iyy="2e-08" iyz="-1e-08" izz="3e-08"/>
+    <inertia ixx="0.0" ixy="0.0" ixz="0.0" iyy="0.0" iyz="-0.0" izz="0.0"/>
   </inertial>
   <visual>
@@ -766,7 +766,7 @@
 <link name="wheel_roller1_3_1">
   <inertial>
-    <origin rpy="0 0 0" xyz="1.8441451409001441e-07 4.051678663199998e-07 3.016277917988752e-07"/>
-    <mass value="0.002562325630105993"/>
-    <inertia ixx="1e-07" ixy="-1e-08" ixz="-1e-08" iyy="9e-08" iyz="1e-08" izz="1e-07"/>
+    <origin rpy="0 0 0" xyz="1.844145140969533e-07 4.051678663199998e-07 3.016277917988752e-07"/>
+    <mass value="0.002562325630105992"/>
+    <inertia ixx="0.0" ixy="-0.0" ixz="-0.0" iyy="0.0" iyz="0.0" izz="0.0"/>
   </inertial>
   <visual>
@@ -788,5 +788,5 @@
     <origin rpy="0 0 0" xyz="-2.1064077822263716e-08 -4.608225134400401e-07 -9.66543238570261e-08"/>
     <mass value="0.0012011377071081556"/>
-    <inertia ixx="2e-08" ixy="-0.0" ixz="1e-08" iyy="3e-08" iyz="0.0" izz="3e-08"/>
+    <inertia ixx="0.0" ixy="-0.0" ixz="0.0" iyy="0.0" iyz="0.0" izz="0.0"/>
   </inertial>
   <visual>
@@ -808,5 +808,5 @@
     <origin rpy="0 0 0" xyz="-4.80340058631179e-07 2.0996169394077446e-07 7.806477175797966e-08"/>
     <mass value="0.002562325630106023"/>
-    <inertia ixx="1.1e-07" ixy="1e-08" ixz="-1e-08" iyy="1e-07" iyz="-1e-08" izz="9e-08"/>
+    <inertia ixx="0.0" ixy="0.0" ixz="-0.0" iyy="0.0" iyz="-0.0" izz="0.0"/>
   </inertial>
   <visual>
@@ -828,5 +828,5 @@
     <origin rpy="0 0 0" xyz="-7.154155730642704e-18 3.19927326214442e-07 -4.949365296977315e-07"/>
     <mass value="0.0012011377071081363"/>
-    <inertia ixx="2e-08" ixy="-0.0" ixz="0.0" iyy="3e-08" iyz="-0.0" izz="3e-08"/>
+    <inertia ixx="0.0" ixy="-0.0" ixz="0.0" iyy="0.0" iyz="-0.0" izz="0.0"/>
   </inertial>
   <visual>
@@ -848,5 +848,5 @@
     <origin rpy="0 0 0" xyz="0.0012986987297723667 0.0005300692565428089 -0.0005302442653455225"/>
     <mass value="0.002562325630106008"/>
-    <inertia ixx="1.1e-07" ixy="1e-08" ixz="-1e-08" iyy="9e-08" iyz="-0.0" izz="9e-08"/>
+    <inertia ixx="0.0" ixy="0.0" ixz="-0.0" iyy="0.0" iyz="-0.0" izz="0.0"/>
   </inertial>
   <visual>
@@ -868,5 +868,5 @@
     <origin rpy="0 0 0" xyz="-2.3788655158923921e-07 -7.835488065321972e-08 -9.665444332396245e-08"/>
     <mass value="0.0012011377071081703"/>
-    <inertia ixx="3e-08" ixy="-0.0" ixz="0.0" iyy="3e-08" iyz="1e-08" izz="3e-08"/>
+    <inertia ixx="0.0" ixy="-0.0" ixz="0.0" iyy="0.0" iyz="0.0" izz="0.0"/>
   </inertial>
   <visual>
@@ -888,5 +888,5 @@
     <origin rpy="0 0 0" xyz="-4.10851908050347e-14 -4.766371183989593e-07 3.016277918058141e-07"/>
     <mass value="0.002562325630106001"/>
-    <inertia ixx="9e-08" ixy="-0.0" ixz="0.0" iyy="1e-07" iyz="-2e-08" izz="1e-07"/>
+    <inertia ixx="0.0" ixy="-0.0" ixz="0.0" iyy="0.0" iyz="-0.0" izz="0.0"/>
   </inertial>
   <visual>
@@ -908,5 +908,5 @@
     <origin rpy="0 0 0" xyz="-2.378865543301023e-07 1.3562872630545897e-09 -1.7636561509652704e-07"/>
     <mass value="0.0012011377071081686"/>
-    <inertia ixx="3e-08" ixy="0.0" ixz="-0.0" iyy="3e-08" iyz="1e-08" izz="3e-08"/>
+    <inertia ixx="0.0" ixy="0.0" ixz="-0.0" iyy="0.0" iyz="0.0" izz="0.0"/>
   </inertial>
   <visual>
@@ -928,5 +928,5 @@
     <origin rpy="0 0 0" xyz="-3.3974599703348596e-07 -2.3573421611966516e-07 6.072436503634648e-08"/>
     <mass value="0.0025623256301060045"/>
-    <inertia ixx="1.1e-07" ixy="-1e-08" ixz="1e-08" iyy="9e-08" iyz="-0.0" izz="9e-08"/>
+    <inertia ixx="0.0" ixy="-0.0" ixz="0.0" iyy="0.0" iyz="-0.0" izz="0.0"/>
   </inertial>
   <visual>
@@ -948,5 +948,5 @@
     <origin rpy="0 0 0" xyz="-1.3354424030533122e-16 -2.732015630807494e-07 9.819211308631504e-08"/>
     <mass value="0.0012011377071081296"/>
-    <inertia ixx="2e-08" ixy="0.0" ixz="-0.0" iyy="3e-08" iyz="-0.0" izz="3e-08"/>
+    <inertia ixx="0.0" ixy="0.0" ixz="-0.0" iyy="0.0" iyz="-0.0" izz="0.0"/>
   </inertial>
   <visual>
@@ -968,5 +968,5 @@
     <origin rpy="0 0 0" xyz="3.685073080017531e-14 2.997996893031041e-07 -4.7480954054775204e-07"/>
     <mass value="0.002562325630106014"/>
-    <inertia ixx="1.1e-07" ixy="1e-08" ixz="-1e-08" iyy="9e-08" iyz="-0.0" izz="9e-08"/>
+    <inertia ixx="0.0" ixy="0.0" ixz="-0.0" iyy="0.0" iyz="-0.0" izz="0.0"/>
   </inertial>
   <visual>
@@ -988,5 +988,5 @@
     <origin rpy="0 0 0" xyz="2.3788655255027602e-07 1.2508064517469109e-07 -3.0008997087965783e-07"/>
     <mass value="0.0012011377071081773"/>
-    <inertia ixx="3e-08" ixy="-0.0" ixz="0.0" iyy="3e-08" iyz="1e-08" izz="3e-08"/>
+    <inertia ixx="0.0" ixy="-0.0" ixz="0.0" iyy="0.0" iyz="0.0" izz="0.0"/>
   </inertial>
   <visual>
@@ -1008,5 +1008,5 @@
     <origin rpy="0 0 0" xyz="4.114070195626596e-14 -4.766371192871377e-07 3.0162779236092563e-07"/>
     <mass value="0.002562325630106015"/>
-    <inertia ixx="9e-08" ixy="0.0" ixz="-0.0" iyy="1e-07" iyz="-2e-08" izz="1e-07"/>
+    <inertia ixx="0.0" ixy="0.0" ixz="-0.0" iyy="0.0" iyz="-0.0" izz="0.0"/>
   </inertial>
   <visual>
@@ -1028,5 +1028,5 @@
     <origin rpy="0 0 0" xyz="2.378865539900965e-07 -7.83548799870859e-08 -9.665444396234069e-08"/>
     <mass value="0.0012011377071081415"/>
-    <inertia ixx="3e-08" ixy="0.0" ixz="-0.0" iyy="3e-08" iyz="1e-08" izz="3e-08"/>
+    <inertia ixx="0.0" ixy="0.0" ixz="-0.0" iyy="0.0" iyz="0.0" izz="0.0"/>
   </inertial>
   <visual>
@@ -1048,5 +1048,5 @@
     <origin rpy="0 0 0" xyz="3.802513859341161e-14 -2.530739275363736e-07 7.806512464930693e-08"/>
     <mass value="0.002562325630106016"/>
-    <inertia ixx="1.1e-07" ixy="-1e-08" ixz="1e-08" iyy="9e-08" iyz="-0.0" izz="9e-08"/>
+    <inertia ixx="0.0" ixy="-0.0" ixz="0.0" iyy="0.0" iyz="-0.0" izz="0.0"/>
   </inertial>
   <visual>
@@ -1068,5 +1068,5 @@
     <origin rpy="0 0 0" xyz="-1.1343589581547242e-08 -1.5996360108044838e-07 -4.949366529324872e-07"/>
     <mass value="0.0012011377071081515"/>
-    <inertia ixx="3e-08" ixy="1e-08" ixz="0.0" iyy="2e-08" iyz="0.0" izz="3e-08"/>
+    <inertia ixx="0.0" ixy="0.0" ixz="0.0" iyy="0.0" iyz="0.0" izz="0.0"/>
   </inertial>
   <visual>
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