Commit message: feat: create ROS2 metapackage

File: deep_ballbot/deepbb_description/urdf/deep_ballbot.xacro (robot description, xacro)
@@ -1,7 +1,7 @@
 <?xml version="1.0" ?>
 <robot name="deep_ballbot" xmlns:xacro="http://www.ros.org/wiki/xacro">
-<xacro:include filename="$(find deep_ballbot)/urdf/materials.xacro" />
-<xacro:include filename="$(find deep_ballbot)/urdf/deep_ballbot.trans" />
-<xacro:include filename="$(find deep_ballbot)/urdf/deep_ballbot.gazebo" />
+<xacro:include filename="$(find deepbb_description)/urdf/materials.xacro" />
+<xacro:include filename="$(find deepbb_description)/urdf/deep_ballbot.trans" />
+<xacro:include filename="$(find deepbb_description)/urdf/deep_ballbot.gazebo" />
 <link name="base_link">
   <inertial>
@@ -13,5 +13,5 @@
     <origin rpy="0 0 0" xyz="0 0 0"/>
     <geometry>
-      <mesh filename="file://$(find deep_ballbot)/meshes/base_link.stl" scale="0.001 0.001 0.001"/>
+      <mesh filename="file://$(find deepbb_description)/meshes/base_link.stl" scale="0.001 0.001 0.001"/>
     </geometry>
     <material name="silver"/>
@@ -20,5 +20,5 @@
     <origin rpy="0 0 0" xyz="0 0 0"/>
     <geometry>
-      <mesh filename="file://$(find deep_ballbot)/meshes/base_link.stl" scale="0.001 0.001 0.001"/>
+      <mesh filename="file://$(find deepbb_description)/meshes/base_link.stl" scale="0.001 0.001 0.001"/>
     </geometry>
   </collision>
@@ -33,5 +33,5 @@
     <origin rpy="0 0 0" xyz="-0.0 -0.0 -0.040825"/>
     <geometry>
-      <mesh filename="file://$(find deep_ballbot)/meshes/base_shell1_1.stl" scale="0.001 0.001 0.001"/>
+      <mesh filename="file://$(find deepbb_description)/meshes/base_shell1_1.stl" scale="0.001 0.001 0.001"/>
     </geometry>
     <material name="silver"/>
@@ -40,5 +40,5 @@
     <origin rpy="0 0 0" xyz="-0.0 -0.0 -0.040825"/>
     <geometry>
-      <mesh filename="file://$(find deep_ballbot)/meshes/base_shell1_1.stl" scale="0.001 0.001 0.001"/>
+      <mesh filename="file://$(find deepbb_description)/meshes/base_shell1_1.stl" scale="0.001 0.001 0.001"/>
     </geometry>
   </collision>
@@ -53,5 +53,5 @@
     <origin rpy="0 0 0" xyz="-0.0 -0.0 -0.040825"/>
     <geometry>
-      <mesh filename="file://$(find deep_ballbot)/meshes/base_shell2_1.stl" scale="0.001 0.001 0.001"/>
+      <mesh filename="file://$(find deepbb_description)/meshes/base_shell2_1.stl" scale="0.001 0.001 0.001"/>
     </geometry>
     <material name="silver"/>
@@ -60,5 +60,5 @@
     <origin rpy="0 0 0" xyz="-0.0 -0.0 -0.040825"/>
     <geometry>
-      <mesh filename="file://$(find deep_ballbot)/meshes/base_shell2_1.stl" scale="0.001 0.001 0.001"/>
+      <mesh filename="file://$(find deepbb_description)/meshes/base_shell2_1.stl" scale="0.001 0.001 0.001"/>
     </geometry>
   </collision>
@@ -73,5 +73,5 @@
     <origin rpy="0 0 0" xyz="-0.0 -0.0 -0.040825"/>
     <geometry>
-      <mesh filename="file://$(find deep_ballbot)/meshes/base_shell3_1.stl" scale="0.001 0.001 0.001"/>
+      <mesh filename="file://$(find deepbb_description)/meshes/base_shell3_1.stl" scale="0.001 0.001 0.001"/>
     </geometry>
     <material name="silver"/>
@@ -80,5 +80,5 @@
     <origin rpy="0 0 0" xyz="-0.0 -0.0 -0.040825"/>
     <geometry>
-      <mesh filename="file://$(find deep_ballbot)/meshes/base_shell3_1.stl" scale="0.001 0.001 0.001"/>
+      <mesh filename="file://$(find deepbb_description)/meshes/base_shell3_1.stl" scale="0.001 0.001 0.001"/>
     </geometry>
   </collision>
@@ -93,5 +93,5 @@
     <origin rpy="0 0 0" xyz="-0.040768 0.044631 -0.085825"/>
     <geometry>
-      <mesh filename="file://$(find deep_ballbot)/meshes/base_plate2_1.stl" scale="0.001 0.001 0.001"/>
+      <mesh filename="file://$(find deepbb_description)/meshes/base_plate2_1.stl" scale="0.001 0.001 0.001"/>
     </geometry>
     <material name="silver"/>
@@ -100,5 +100,5 @@
     <origin rpy="0 0 0" xyz="-0.040768 0.044631 -0.085825"/>
     <geometry>
-      <mesh filename="file://$(find deep_ballbot)/meshes/base_plate2_1.stl" scale="0.001 0.001 0.001"/>
+      <mesh filename="file://$(find deepbb_description)/meshes/base_plate2_1.stl" scale="0.001 0.001 0.001"/>
     </geometry>
   </collision>
@@ -113,5 +113,5 @@
     <origin rpy="0 0 0" xyz="-0.018268 -0.057622 -0.085825"/>
     <geometry>
-      <mesh filename="file://$(find deep_ballbot)/meshes/base_plate3_1.stl" scale="0.001 0.001 0.001"/>
+      <mesh filename="file://$(find deepbb_description)/meshes/base_plate3_1.stl" scale="0.001 0.001 0.001"/>
     </geometry>
     <material name="silver"/>
@@ -120,5 +120,5 @@
     <origin rpy="0 0 0" xyz="-0.018268 -0.057622 -0.085825"/>
     <geometry>
-      <mesh filename="file://$(find deep_ballbot)/meshes/base_plate3_1.stl" scale="0.001 0.001 0.001"/>
+      <mesh filename="file://$(find deepbb_description)/meshes/base_plate3_1.stl" scale="0.001 0.001 0.001"/>
     </geometry>
   </collision>
@@ -133,5 +133,5 @@
     <origin rpy="0 0 0" xyz="0.023921 0.013811 -0.088825"/>
     <geometry>
-      <mesh filename="file://$(find deep_ballbot)/meshes/vertical_bay1_1.stl" scale="0.001 0.001 0.001"/>
+      <mesh filename="file://$(find deepbb_description)/meshes/vertical_bay1_1.stl" scale="0.001 0.001 0.001"/>
     </geometry>
     <material name="silver"/>
@@ -140,5 +140,5 @@
     <origin rpy="0 0 0" xyz="0.023921 0.013811 -0.088825"/>
     <geometry>
-      <mesh filename="file://$(find deep_ballbot)/meshes/vertical_bay1_1.stl" scale="0.001 0.001 0.001"/>
+      <mesh filename="file://$(find deepbb_description)/meshes/vertical_bay1_1.stl" scale="0.001 0.001 0.001"/>
     </geometry>
   </collision>
@@ -153,5 +153,5 @@
     <origin rpy="0 0 0" xyz="-0.023921 0.013811 -0.088825"/>
     <geometry>
-      <mesh filename="file://$(find deep_ballbot)/meshes/vertical_bay2_1.stl" scale="0.001 0.001 0.001"/>
+      <mesh filename="file://$(find deepbb_description)/meshes/vertical_bay2_1.stl" scale="0.001 0.001 0.001"/>
     </geometry>
     <material name="silver"/>
@@ -160,5 +160,5 @@
     <origin rpy="0 0 0" xyz="-0.023921 0.013811 -0.088825"/>
     <geometry>
-      <mesh filename="file://$(find deep_ballbot)/meshes/vertical_bay2_1.stl" scale="0.001 0.001 0.001"/>
+      <mesh filename="file://$(find deepbb_description)/meshes/vertical_bay2_1.stl" scale="0.001 0.001 0.001"/>
     </geometry>
   </collision>
@@ -173,5 +173,5 @@
     <origin rpy="0 0 0" xyz="-0.0 -0.027622 -0.088825"/>
     <geometry>
-      <mesh filename="file://$(find deep_ballbot)/meshes/vertical_bay3_1.stl" scale="0.001 0.001 0.001"/>
+      <mesh filename="file://$(find deepbb_description)/meshes/vertical_bay3_1.stl" scale="0.001 0.001 0.001"/>
     </geometry>
     <material name="silver"/>
@@ -180,5 +180,5 @@
     <origin rpy="0 0 0" xyz="-0.0 -0.027622 -0.088825"/>
     <geometry>
-      <mesh filename="file://$(find deep_ballbot)/meshes/vertical_bay3_1.stl" scale="0.001 0.001 0.001"/>
+      <mesh filename="file://$(find deepbb_description)/meshes/vertical_bay3_1.stl" scale="0.001 0.001 0.001"/>
     </geometry>
   </collision>
@@ -193,5 +193,5 @@
     <origin rpy="0 0 0" xyz="0.0 0.047631 -0.159825"/>
     <geometry>
-      <mesh filename="file://$(find deep_ballbot)/meshes/breadboard_1.stl" scale="0.001 0.001 0.001"/>
+      <mesh filename="file://$(find deepbb_description)/meshes/breadboard_1.stl" scale="0.001 0.001 0.001"/>
     </geometry>
     <material name="silver"/>
@@ -200,5 +200,5 @@
     <origin rpy="0 0 0" xyz="0.0 0.047631 -0.159825"/>
     <geometry>
-      <mesh filename="file://$(find deep_ballbot)/meshes/breadboard_1.stl" scale="0.001 0.001 0.001"/>
+      <mesh filename="file://$(find deepbb_description)/meshes/breadboard_1.stl" scale="0.001 0.001 0.001"/>
     </geometry>
   </collision>
@@ -213,5 +213,5 @@
     <origin rpy="0 0 0" xyz="0.0 -0.0105 -0.159825"/>
     <geometry>
-      <mesh filename="file://$(find deep_ballbot)/meshes/rasbperry_pi_1.stl" scale="0.001 0.001 0.001"/>
+      <mesh filename="file://$(find deepbb_description)/meshes/rasbperry_pi_1.stl" scale="0.001 0.001 0.001"/>
     </geometry>
     <material name="silver"/>
@@ -220,5 +220,5 @@
     <origin rpy="0 0 0" xyz="0.0 -0.0105 -0.159825"/>
     <geometry>
-      <mesh filename="file://$(find deep_ballbot)/meshes/rasbperry_pi_1.stl" scale="0.001 0.001 0.001"/>
+      <mesh filename="file://$(find deepbb_description)/meshes/rasbperry_pi_1.stl" scale="0.001 0.001 0.001"/>
     </geometry>
   </collision>
@@ -233,5 +233,5 @@
     <origin rpy="0 0 0" xyz="0.046487 -0.026839 -0.072881"/>
     <geometry>
-      <mesh filename="file://$(find deep_ballbot)/meshes/motor_mount1_1.stl" scale="0.001 0.001 0.001"/>
+      <mesh filename="file://$(find deepbb_description)/meshes/motor_mount1_1.stl" scale="0.001 0.001 0.001"/>
     </geometry>
     <material name="silver"/>
@@ -240,5 +240,5 @@
     <origin rpy="0 0 0" xyz="0.046487 -0.026839 -0.072881"/>
     <geometry>
-      <mesh filename="file://$(find deep_ballbot)/meshes/motor_mount1_1.stl" scale="0.001 0.001 0.001"/>
+      <mesh filename="file://$(find deepbb_description)/meshes/motor_mount1_1.stl" scale="0.001 0.001 0.001"/>
     </geometry>
   </collision>
@@ -253,5 +253,5 @@
     <origin rpy="0 0 0" xyz="-0.0 0.053678 -0.072881"/>
     <geometry>
-      <mesh filename="file://$(find deep_ballbot)/meshes/motor_mount2_1.stl" scale="0.001 0.001 0.001"/>
+      <mesh filename="file://$(find deepbb_description)/meshes/motor_mount2_1.stl" scale="0.001 0.001 0.001"/>
     </geometry>
     <material name="silver"/>
@@ -260,5 +260,5 @@
     <origin rpy="0 0 0" xyz="-0.0 0.053678 -0.072881"/>
     <geometry>
-      <mesh filename="file://$(find deep_ballbot)/meshes/motor_mount2_1.stl" scale="0.001 0.001 0.001"/>
+      <mesh filename="file://$(find deepbb_description)/meshes/motor_mount2_1.stl" scale="0.001 0.001 0.001"/>
     </geometry>
   </collision>
@@ -273,5 +273,5 @@
     <origin rpy="0 0 0" xyz="-0.046487 -0.026839 -0.072881"/>
     <geometry>
-      <mesh filename="file://$(find deep_ballbot)/meshes/motor_mount3_1.stl" scale="0.001 0.001 0.001"/>
+      <mesh filename="file://$(find deepbb_description)/meshes/motor_mount3_1.stl" scale="0.001 0.001 0.001"/>
     </geometry>
     <material name="silver"/>
@@ -280,5 +280,5 @@
     <origin rpy="0 0 0" xyz="-0.046487 -0.026839 -0.072881"/>
     <geometry>
-      <mesh filename="file://$(find deep_ballbot)/meshes/motor_mount3_1.stl" scale="0.001 0.001 0.001"/>
+      <mesh filename="file://$(find deepbb_description)/meshes/motor_mount3_1.stl" scale="0.001 0.001 0.001"/>
     </geometry>
   </collision>
@@ -293,5 +293,5 @@
     <origin rpy="0 0 0" xyz="0.026519 0.015311 -0.121325"/>
     <geometry>
-      <mesh filename="file://$(find deep_ballbot)/meshes/arduino_mount1_1.stl" scale="0.001 0.001 0.001"/>
+      <mesh filename="file://$(find deepbb_description)/meshes/arduino_mount1_1.stl" scale="0.001 0.001 0.001"/>
     </geometry>
     <material name="silver"/>
@@ -300,5 +300,5 @@
     <origin rpy="0 0 0" xyz="0.026519 0.015311 -0.121325"/>
     <geometry>
-      <mesh filename="file://$(find deep_ballbot)/meshes/arduino_mount1_1.stl" scale="0.001 0.001 0.001"/>
+      <mesh filename="file://$(find deepbb_description)/meshes/arduino_mount1_1.stl" scale="0.001 0.001 0.001"/>
     </geometry>
   </collision>
@@ -313,5 +313,5 @@
     <origin rpy="0 0 0" xyz="-0.026519 0.015311 -0.121325"/>
     <geometry>
-      <mesh filename="file://$(find deep_ballbot)/meshes/arduino_mount2_1.stl" scale="0.001 0.001 0.001"/>
+      <mesh filename="file://$(find deepbb_description)/meshes/arduino_mount2_1.stl" scale="0.001 0.001 0.001"/>
     </geometry>
     <material name="silver"/>
@@ -320,5 +320,5 @@
     <origin rpy="0 0 0" xyz="-0.026519 0.015311 -0.121325"/>
     <geometry>
-      <mesh filename="file://$(find deep_ballbot)/meshes/arduino_mount2_1.stl" scale="0.001 0.001 0.001"/>
+      <mesh filename="file://$(find deepbb_description)/meshes/arduino_mount2_1.stl" scale="0.001 0.001 0.001"/>
     </geometry>
   </collision>
@@ -333,5 +333,5 @@
     <origin rpy="0 0 0" xyz="-0.0 -0.030622 -0.121325"/>
     <geometry>
-      <mesh filename="file://$(find deep_ballbot)/meshes/arduino_mount3_1.stl" scale="0.001 0.001 0.001"/>
+      <mesh filename="file://$(find deepbb_description)/meshes/arduino_mount3_1.stl" scale="0.001 0.001 0.001"/>
     </geometry>
     <material name="silver"/>
@@ -340,5 +340,5 @@
     <origin rpy="0 0 0" xyz="-0.0 -0.030622 -0.121325"/>
     <geometry>
-      <mesh filename="file://$(find deep_ballbot)/meshes/arduino_mount3_1.stl" scale="0.001 0.001 0.001"/>
+      <mesh filename="file://$(find deepbb_description)/meshes/arduino_mount3_1.stl" scale="0.001 0.001 0.001"/>
     </geometry>
   </collision>
@@ -353,5 +353,5 @@
     <origin rpy="0 0 0" xyz="0.047078 -0.010299 -0.112825"/>
     <geometry>
-      <mesh filename="file://$(find deep_ballbot)/meshes/arduino1_1.stl" scale="0.001 0.001 0.001"/>
+      <mesh filename="file://$(find deepbb_description)/meshes/arduino1_1.stl" scale="0.001 0.001 0.001"/>
     </geometry>
     <material name="silver"/>
@@ -360,5 +360,5 @@
     <origin rpy="0 0 0" xyz="0.047078 -0.010299 -0.112825"/>
     <geometry>
-      <mesh filename="file://$(find deep_ballbot)/meshes/arduino1_1.stl" scale="0.001 0.001 0.001"/>
+      <mesh filename="file://$(find deepbb_description)/meshes/arduino1_1.stl" scale="0.001 0.001 0.001"/>
     </geometry>
   </collision>
@@ -373,5 +373,5 @@
     <origin rpy="0 0 0" xyz="-0.01462 0.04592 -0.112825"/>
     <geometry>
-      <mesh filename="file://$(find deep_ballbot)/meshes/arduino2_1.stl" scale="0.001 0.001 0.001"/>
+      <mesh filename="file://$(find deepbb_description)/meshes/arduino2_1.stl" scale="0.001 0.001 0.001"/>
     </geometry>
     <material name="silver"/>
@@ -380,5 +380,5 @@
     <origin rpy="0 0 0" xyz="-0.01462 0.04592 -0.112825"/>
     <geometry>
-      <mesh filename="file://$(find deep_ballbot)/meshes/arduino2_1.stl" scale="0.001 0.001 0.001"/>
+      <mesh filename="file://$(find deepbb_description)/meshes/arduino2_1.stl" scale="0.001 0.001 0.001"/>
     </geometry>
   </collision>
@@ -393,5 +393,5 @@
     <origin rpy="0 0 0" xyz="-0.032458 -0.035622 -0.112825"/>
     <geometry>
-      <mesh filename="file://$(find deep_ballbot)/meshes/arduino3_1.stl" scale="0.001 0.001 0.001"/>
+      <mesh filename="file://$(find deepbb_description)/meshes/arduino3_1.stl" scale="0.001 0.001 0.001"/>
     </geometry>
     <material name="silver"/>
@@ -400,5 +400,5 @@
     <origin rpy="0 0 0" xyz="-0.032458 -0.035622 -0.112825"/>
     <geometry>
-      <mesh filename="file://$(find deep_ballbot)/meshes/arduino3_1.stl" scale="0.001 0.001 0.001"/>
+      <mesh filename="file://$(find deepbb_description)/meshes/arduino3_1.stl" scale="0.001 0.001 0.001"/>
     </geometry>
   </collision>
@@ -413,5 +413,5 @@
     <origin rpy="0 0 0" xyz="0.051386 -0.029667 -0.067224"/>
     <geometry>
-      <mesh filename="file://$(find deep_ballbot)/meshes/motor_stator1_1.stl" scale="0.001 0.001 0.001"/>
+      <mesh filename="file://$(find deepbb_description)/meshes/motor_stator1_1.stl" scale="0.001 0.001 0.001"/>
     </geometry>
     <material name="silver"/>
@@ -420,5 +420,5 @@
     <origin rpy="0 0 0" xyz="0.051386 -0.029667 -0.067224"/>
     <geometry>
-      <mesh filename="file://$(find deep_ballbot)/meshes/motor_stator1_1.stl" scale="0.001 0.001 0.001"/>
+      <mesh filename="file://$(find deepbb_description)/meshes/motor_stator1_1.stl" scale="0.001 0.001 0.001"/>
     </geometry>
   </collision>
@@ -433,5 +433,5 @@
     <origin rpy="0 0 0" xyz="-0.0 0.059335 -0.067224"/>
     <geometry>
-      <mesh filename="file://$(find deep_ballbot)/meshes/motor_stator2_1.stl" scale="0.001 0.001 0.001"/>
+      <mesh filename="file://$(find deepbb_description)/meshes/motor_stator2_1.stl" scale="0.001 0.001 0.001"/>
     </geometry>
     <material name="silver"/>
@@ -440,5 +440,5 @@
     <origin rpy="0 0 0" xyz="-0.0 0.059335 -0.067224"/>
     <geometry>
-      <mesh filename="file://$(find deep_ballbot)/meshes/motor_stator2_1.stl" scale="0.001 0.001 0.001"/>
+      <mesh filename="file://$(find deepbb_description)/meshes/motor_stator2_1.stl" scale="0.001 0.001 0.001"/>
     </geometry>
   </collision>
@@ -453,5 +453,5 @@
     <origin rpy="0 0 0" xyz="-0.051386 -0.029667 -0.067224"/>
     <geometry>
-      <mesh filename="file://$(find deep_ballbot)/meshes/motor_stator3_1.stl" scale="0.001 0.001 0.001"/>
+      <mesh filename="file://$(find deepbb_description)/meshes/motor_stator3_1.stl" scale="0.001 0.001 0.001"/>
     </geometry>
     <material name="silver"/>
@@ -460,5 +460,5 @@
     <origin rpy="0 0 0" xyz="-0.051386 -0.029667 -0.067224"/>
     <geometry>
-      <mesh filename="file://$(find deep_ballbot)/meshes/motor_stator3_1.stl" scale="0.001 0.001 0.001"/>
+      <mesh filename="file://$(find deepbb_description)/meshes/motor_stator3_1.stl" scale="0.001 0.001 0.001"/>
     </geometry>
   </collision>
@@ -473,5 +473,5 @@
     <origin rpy="0 0 0" xyz="0.041588 -0.024011 -0.047426"/>
     <geometry>
-      <mesh filename="file://$(find deep_ballbot)/meshes/motor_rotor1_1.stl" scale="0.001 0.001 0.001"/>
+      <mesh filename="file://$(find deepbb_description)/meshes/motor_rotor1_1.stl" scale="0.001 0.001 0.001"/>
     </geometry>
     <material name="silver"/>
@@ -480,5 +480,5 @@
     <origin rpy="0 0 0" xyz="0.041588 -0.024011 -0.047426"/>
     <geometry>
-      <mesh filename="file://$(find deep_ballbot)/meshes/motor_rotor1_1.stl" scale="0.001 0.001 0.001"/>
+      <mesh filename="file://$(find deepbb_description)/meshes/motor_rotor1_1.stl" scale="0.001 0.001 0.001"/>
     </geometry>
   </collision>
@@ -493,5 +493,5 @@
     <origin rpy="0 0 0" xyz="-0.0 0.048021 -0.047426"/>
     <geometry>
-      <mesh filename="file://$(find deep_ballbot)/meshes/motor_rotor2_1.stl" scale="0.001 0.001 0.001"/>
+      <mesh filename="file://$(find deepbb_description)/meshes/motor_rotor2_1.stl" scale="0.001 0.001 0.001"/>
     </geometry>
     <material name="silver"/>
@@ -500,5 +500,5 @@
     <origin rpy="0 0 0" xyz="-0.0 0.048021 -0.047426"/>
     <geometry>
-      <mesh filename="file://$(find deep_ballbot)/meshes/motor_rotor2_1.stl" scale="0.001 0.001 0.001"/>
+      <mesh filename="file://$(find deepbb_description)/meshes/motor_rotor2_1.stl" scale="0.001 0.001 0.001"/>
     </geometry>
   </collision>
@@ -513,5 +513,5 @@
     <origin rpy="0 0 0" xyz="-0.041588 -0.024011 -0.047426"/>
     <geometry>
-      <mesh filename="file://$(find deep_ballbot)/meshes/motor_rotor3_1.stl" scale="0.001 0.001 0.001"/>
+      <mesh filename="file://$(find deepbb_description)/meshes/motor_rotor3_1.stl" scale="0.001 0.001 0.001"/>
     </geometry>
     <material name="silver"/>
@@ -520,5 +520,5 @@
     <origin rpy="0 0 0" xyz="-0.041588 -0.024011 -0.047426"/>
     <geometry>
-      <mesh filename="file://$(find deep_ballbot)/meshes/motor_rotor3_1.stl" scale="0.001 0.001 0.001"/>
+      <mesh filename="file://$(find deepbb_description)/meshes/motor_rotor3_1.stl" scale="0.001 0.001 0.001"/>
     </geometry>
   </collision>
@@ -533,5 +533,5 @@
     <origin rpy="0 0 0" xyz="0.05261 -0.030375 -0.034698"/>
     <geometry>
-      <mesh filename="file://$(find deep_ballbot)/meshes/wheel_body1_1.stl" scale="0.001 0.001 0.001"/>
+      <mesh filename="file://$(find deepbb_description)/meshes/wheel_body1_1.stl" scale="0.001 0.001 0.001"/>
     </geometry>
     <material name="silver"/>
@@ -540,5 +540,5 @@
     <origin rpy="0 0 0" xyz="0.05261 -0.030375 -0.034698"/>
     <geometry>
-      <mesh filename="file://$(find deep_ballbot)/meshes/wheel_body1_1.stl" scale="0.001 0.001 0.001"/>
+      <mesh filename="file://$(find deepbb_description)/meshes/wheel_body1_1.stl" scale="0.001 0.001 0.001"/>
     </geometry>
   </collision>
@@ -553,5 +553,5 @@
     <origin rpy="0 0 0" xyz="-0.0 0.060749 -0.034698"/>
     <geometry>
-      <mesh filename="file://$(find deep_ballbot)/meshes/wheel_body2_1.stl" scale="0.001 0.001 0.001"/>
+      <mesh filename="file://$(find deepbb_description)/meshes/wheel_body2_1.stl" scale="0.001 0.001 0.001"/>
     </geometry>
     <material name="silver"/>
@@ -560,5 +560,5 @@
     <origin rpy="0 0 0" xyz="-0.0 0.060749 -0.034698"/>
     <geometry>
-      <mesh filename="file://$(find deep_ballbot)/meshes/wheel_body2_1.stl" scale="0.001 0.001 0.001"/>
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