Commit message: fix: modify omniwheel inertias + damping for sim stability

File: deepbb_description/urdf/deep_ballbot_new.xacro (robot description, xacro)
@@ -1,7 +1,7 @@
 <?xml version="1.0" ?>
 <robot name="deep_ballbot" xmlns:xacro="http://www.ros.org/wiki/xacro">
-<xacro:include filename="$(find deepbb_description)/urdf/materials.xacro" />
-<xacro:include filename="$(find deepbb_description)/urdf/deep_ballbot.trans" />
-<xacro:include filename="$(find deepbb_description)/urdf/deep_ballbot.gazebo" />
+<xacro:include filename="$(find deep_ballbot_description)/urdf/materials.xacro" />
+<xacro:include filename="$(find deep_ballbot_description)/urdf/deep_ballbot.trans" />
+<xacro:include filename="$(find deep_ballbot_description)/urdf/deep_ballbot.gazebo" />
 <link name="base_link">
   <inertial>
@@ -15,5 +15,5 @@
       <mesh filename="file://$(find deepbb_description)/meshes/base_link.stl" scale="0.001 0.001 0.001"/>
     </geometry>
-    <material name="black"/>
+    <material name="grey"/>
   </visual>
   <collision>
@@ -35,5 +35,5 @@
       <mesh filename="file://$(find deepbb_description)/meshes/base_shell1_1.stl" scale="0.001 0.001 0.001"/>
     </geometry>
-    <material name="white"/>
+    <material name="grey"/>
   </visual>
   <collision>
@@ -55,5 +55,5 @@
       <mesh filename="file://$(find deepbb_description)/meshes/base_shell2_1.stl" scale="0.001 0.001 0.001"/>
     </geometry>
-    <material name="white"/>
+    <material name="grey"/>
   </visual>
   <collision>
@@ -75,5 +75,5 @@
       <mesh filename="file://$(find deepbb_description)/meshes/base_shell3_1.stl" scale="0.001 0.001 0.001"/>
     </geometry>
-    <material name="white"/>
+    <material name="grey"/>
   </visual>
   <collision>
@@ -195,5 +195,5 @@
       <mesh filename="file://$(find deepbb_description)/meshes/breadboard_1.stl" scale="0.001 0.001 0.001"/>
     </geometry>
-    <material name="white"/>
+    <material name="grey"/>
   </visual>
   <collision>
@@ -215,5 +215,5 @@
       <mesh filename="file://$(find deepbb_description)/meshes/rasbperry_pi_1.stl" scale="0.001 0.001 0.001"/>
     </geometry>
-    <material name="black"/>
+    <material name="grey"/>
   </visual>
   <collision>
@@ -355,5 +355,5 @@
       <mesh filename="file://$(find deepbb_description)/meshes/arduino1_1.stl" scale="0.001 0.001 0.001"/>
     </geometry>
-    <material name="black"/>
+    <material name="grey"/>
   </visual>
   <collision>
@@ -375,5 +375,5 @@
       <mesh filename="file://$(find deepbb_description)/meshes/arduino2_1.stl" scale="0.001 0.001 0.001"/>
     </geometry>
-    <material name="black"/>
+    <material name="grey"/>
   </visual>
   <collision>
@@ -395,5 +395,5 @@
       <mesh filename="file://$(find deepbb_description)/meshes/arduino3_1.stl" scale="0.001 0.001 0.001"/>
     </geometry>
-    <material name="black"/>
+    <material name="grey"/>
   </visual>
   <collision>
@@ -415,5 +415,5 @@
       <mesh filename="file://$(find deepbb_description)/meshes/motor_stator1_1.stl" scale="0.001 0.001 0.001"/>
     </geometry>
-    <material name="black"/>
+    <material name="grey"/>
   </visual>
   <collision>
@@ -435,5 +435,5 @@
       <mesh filename="file://$(find deepbb_description)/meshes/motor_stator2_1.stl" scale="0.001 0.001 0.001"/>
     </geometry>
-    <material name="black"/>
+    <material name="grey"/>
   </visual>
   <collision>
@@ -455,5 +455,5 @@
       <mesh filename="file://$(find deepbb_description)/meshes/motor_stator3_1.stl" scale="0.001 0.001 0.001"/>
     </geometry>
-    <material name="black"/>
+    <material name="grey"/>
   </visual>
   <collision>
@@ -475,5 +475,5 @@
       <mesh filename="file://$(find deepbb_description)/meshes/motor_rotor1_1.stl" scale="0.001 0.001 0.001"/>
     </geometry>
-    <material name="black"/>
+    <material name="grey"/>
   </visual>
   <collision>
@@ -495,5 +495,5 @@
       <mesh filename="file://$(find deepbb_description)/meshes/motor_rotor2_1.stl" scale="0.001 0.001 0.001"/>
     </geometry>
-    <material name="black"/>
+    <material name="grey"/>
   </visual>
   <collision>
@@ -515,5 +515,5 @@
       <mesh filename="file://$(find deepbb_description)/meshes/motor_rotor3_1.stl" scale="0.001 0.001 0.001"/>
     </geometry>
-    <material name="black"/>
+    <material name="grey"/>
   </visual>
   <collision>
@@ -535,5 +535,5 @@
       <mesh filename="file://$(find deepbb_description)/meshes/wheel_body1_1.stl" scale="0.001 0.001 0.001"/>
     </geometry>
-    <material name="white"/>
+    <material name="grey"/>
   </visual>
   <collision>
@@ -555,5 +555,5 @@
       <mesh filename="file://$(find deepbb_description)/meshes/wheel_body2_1.stl" scale="0.001 0.001 0.001"/>
     </geometry>
-    <material name="white"/>
+    <material name="grey"/>
   </visual>
   <collision>
@@ -575,5 +575,5 @@
       <mesh filename="file://$(find deepbb_description)/meshes/wheel_body3_1.stl" scale="0.001 0.001 0.001"/>
     </geometry>
-    <material name="white"/>
+    <material name="grey"/>
   </visual>
   <collision>
@@ -1315,5 +1315,5 @@
       <mesh filename="file://$(find deepbb_description)/meshes/simplefocshield1_1.stl" scale="0.001 0.001 0.001"/>
     </geometry>
-    <material name="black"/>
+    <material name="grey"/>
   </visual>
   <collision>
@@ -1335,5 +1335,5 @@
       <mesh filename="file://$(find deepbb_description)/meshes/simplefocshield2_1.stl" scale="0.001 0.001 0.001"/>
     </geometry>
-    <material name="black"/>
+    <material name="grey"/>
   </visual>
   <collision>
@@ -1355,5 +1355,5 @@
       <mesh filename="file://$(find deepbb_description)/meshes/simplefocshield3_1.stl" scale="0.001 0.001 0.001"/>
     </geometry>
-    <material name="black"/>
+    <material name="grey"/>
   </visual>
   <collision>
@@ -1395,5 +1395,5 @@
       <mesh filename="file://$(find deepbb_description)/meshes/top_plate_1.stl" scale="0.001 0.001 0.001"/>
     </geometry>
-    <material name="white"/>
+    <material name="grey"/>
   </visual>
   <collision>
@@ -1415,5 +1415,5 @@
       <mesh filename="file://$(find deepbb_description)/meshes/arduino_nano_1.stl" scale="0.001 0.001 0.001"/>
     </geometry>
-    <material name="black"/>
+    <material name="grey"/>
   </visual>
   <collision>
@@ -1572,5 +1572,4 @@
   <child link="wheel_roller1_2_1"/>
   <axis xyz="0.5 0.866025 0.0"/>
-  <dynamics damping="0.0"/>
 </joint>
 <joint name="Rev2" type="continuous">
@@ -1579,5 +1578,4 @@
   <child link="wheel_roller1_4_1"/>
   <axis xyz="-0.126826 -0.926777 -0.353553"/>
-  <dynamics damping="0.0"/>
 </joint>
 <joint name="Rev3" type="continuous">
@@ -1586,5 +1584,4 @@
   <child link="wheel_roller1_9_1"/>
   <axis xyz="0.28033 -0.739199 -0.612372"/>
-  <dynamics damping="0.0"/>
 </joint>
 <joint name="Rev4" type="continuous">
@@ -1593,5 +1590,4 @@
   <child link="wheel_roller1_7_1"/>
   <axis xyz="0.612372 -0.353553 -0.707107"/>
-  <dynamics damping="0.0"/>
 </joint>
 <joint name="Rev5" type="continuous">
@@ -1600,5 +1596,4 @@
   <child link="wheel_roller1_12_1"/>
   <axis xyz="-0.78033 -0.126826 0.612372"/>
-  <dynamics damping="0.0"/>
 </joint>
 <joint name="Rev6" type="continuous">
@@ -1607,5 +1602,4 @@
   <child link="wheel_roller1_5_1"/>
   <axis xyz="0.739199 0.573223 -0.353553"/>
-  <dynamics damping="0.0"/>
 </joint>
 <joint name="Rev7" type="continuous">
@@ -1614,5 +1608,4 @@
   <child link="wheel_roller1_10_1"/>
   <axis xyz="-0.5 -0.866025 0.0"/>
-  <dynamics damping="0.0"/>
 </joint>
 <joint name="Rev8" type="continuous">
@@ -1621,5 +1614,4 @@
   <child link="wheel_roller1_6_1"/>
   <axis xyz="-0.126826 -0.926777 -0.353553"/>
-  <dynamics damping="0.0"/>
 </joint>
 <joint name="Rev9" type="continuous">
@@ -1628,5 +1620,4 @@
   <child link="wheel_roller1_11_1"/>
   <axis xyz="0.28033 -0.739199 -0.612372"/>
-  <dynamics damping="0.0"/>
 </joint>
 <joint name="Rev10" type="continuous">
@@ -1635,5 +1626,4 @@
   <child link="wheel_roller1_3_1"/>
   <axis xyz="0.612372 -0.353553 -0.707107"/>
-  <dynamics damping="0.0"/>
 </joint>
 <joint name="Rev11" type="continuous">
@@ -1642,5 +1632,4 @@
   <child link="wheel_roller1_8_1"/>
   <axis xyz="0.78033 0.126826 -0.612372"/>
-  <dynamics damping="0.0"/>
 </joint>
 <joint name="Rev12" type="continuous">
@@ -1649,5 +1638,4 @@
   <child link="wheel_roller1_1_1"/>
   <axis xyz="0.739199 0.573223 -0.353553"/>
-  <dynamics damping="0.0"/>
 </joint>
 <joint name="Rev13" type="continuous">
@@ -1656,5 +1644,4 @@
   <child link="wheel_roller2_2_1"/>
   <axis xyz="-1.0 0.0 0.0"/>
-  <dynamics damping="0.0"/>
 </joint>
 <joint name="Rev14" type="continuous">
@@ -1663,5 +1650,4 @@
   <child link="wheel_roller2_4_1"/>
   <axis xyz="0.866025 0.353553 -0.353553"/>
-  <dynamics damping="0.0"/>
 </joint>
 <joint name="Rev15" type="continuous">
@@ -1670,5 +1656,4 @@
   <child link="wheel_roller2_7_1"/>
   <axis xyz="0.5 0.612372 -0.612372"/>
-  <dynamics damping="0.0"/>
 </joint>
 <joint name="Rev16" type="continuous">
@@ -1677,5 +1662,4 @@
   <child link="wheel_roller2_12_1"/>
   <axis xyz="0.0 0.707107 -0.707107"/>
-  <dynamics damping="0.0"/>
 </joint>
 <joint name="Rev17" type="continuous">
@@ -1684,5 +1668,4 @@
   <child link="wheel_roller2_9_1"/>
   <axis xyz="0.5 -0.612372 0.612372"/>
-  <dynamics damping="0.0"/>
 </joint>
 <joint name="Rev18" type="continuous">
@@ -1691,5 +1674,4 @@
   <child link="wheel_roller2_5_1"/>
   <axis xyz="-0.866025 0.353553 -0.353553"/>
-  <dynamics damping="0.0"/>
 </joint>
 <joint name="Rev19" type="continuous">
@@ -1698,5 +1680,4 @@
   <child link="wheel_roller2_10_1"/>
   <axis xyz="1.0 -0.0 0.0"/>
-  <dynamics damping="0.0"/>
 </joint>
 <joint name="Rev20" type="continuous">
@@ -1705,5 +1686,4 @@
   <child link="wheel_roller2_6_1"/>
   <axis xyz="0.866025 0.353553 -0.353553"/>
-  <dynamics damping="0.0"/>
 </joint>
 <joint name="Rev21" type="continuous">
@@ -1712,5 +1692,4 @@
   <child link="wheel_roller2_11_1"/>
   <axis xyz="0.5 0.612372 -0.612372"/>
-  <dynamics damping="0.0"/>
 </joint>
 <joint name="Rev22" type="continuous">
@@ -1719,5 +1698,4 @@
   <child link="wheel_roller2_3_1"/>
   <axis xyz="0.0 0.707107 -0.707107"/>
-  <dynamics damping="0.0"/>
 </joint>
 <joint name="Rev23" type="continuous">
@@ -1726,5 +1704,4 @@
   <child link="wheel_roller2_8_1"/>
   <axis xyz="-0.5 0.612372 -0.612372"/>
-  <dynamics damping="0.0"/>
 </joint>
 <joint name="Rev24" type="continuous">
@@ -1733,5 +1710,4 @@
   <child link="wheel_roller2_1_1"/>
   <axis xyz="-0.866025 0.353553 -0.353553"/>
-  <dynamics damping="0.0"/>
 </joint>
 <joint name="Rev25" type="continuous">
@@ -1740,5 +1716,4 @@
   <child link="wheel_roller3_2_1"/>
   <axis xyz="0.5 -0.866025 0.0"/>
-  <dynamics damping="0.0"/>
 </joint>
 <joint name="Rev26" type="continuous">
@@ -1747,5 +1722,4 @@
   <child link="wheel_roller3_4_1"/>
   <axis xyz="-0.739199 0.573223 -0.353553"/>
-  <dynamics damping="0.0"/>
 </joint>
 <joint name="Rev27" type="continuous">
@@ -1754,5 +1728,4 @@
   <child link="wheel_roller3_9_1"/>
   <axis xyz="-0.78033 0.126826 -0.612372"/>
-  <dynamics damping="0.0"/>
 </joint>
 <joint name="Rev28" type="continuous">
@@ -1761,5 +1734,4 @@
   <child link="wheel_roller3_7_1"/>
   <axis xyz="-0.612372 -0.353553 -0.707107"/>
-  <dynamics damping="0.0"/>
 </joint>
 <joint name="Rev29" type="continuous">
@@ -1768,5 +1740,4 @@
   <child link="wheel_roller3_12_1"/>
   <axis xyz="0.28033 0.739199 0.612372"/>
-  <dynamics damping="0.0"/>
 </joint>
 <joint name="Rev30" type="continuous">
@@ -1775,5 +1746,4 @@
   <child link="wheel_roller3_5_1"/>
   <axis xyz="0.126826 -0.926777 -0.353553"/>
-  <dynamics damping="0.0"/>
 </joint>
 <joint name="Rev31" type="continuous">
@@ -1782,5 +1752,4 @@
   <child link="wheel_roller3_10_1"/>
   <axis xyz="-0.5 0.866025 0.0"/>
-  <dynamics damping="0.0"/>
 </joint>
 <joint name="Rev32" type="continuous">
@@ -1789,5 +1758,4 @@
   <child link="wheel_roller3_6_1"/>
   <axis xyz="-0.739199 0.573223 -0.353553"/>
-  <dynamics damping="0.0"/>
 </joint>
 <joint name="Rev33" type="continuous">
@@ -1796,5 +1764,4 @@
   <child link="wheel_roller3_11_1"/>
   <axis xyz="-0.78033 0.126826 -0.612372"/>
-  <dynamics damping="0.0"/>
 </joint>
 <joint name="Rev34" type="continuous">
@@ -1803,5 +1770,4 @@
   <child link="wheel_roller3_3_1"/>
   <axis xyz="-0.612372 -0.353553 -0.707107"/>
-  <dynamics damping="0.0"/>
 </joint>
 <joint name="Rev35" type="continuous">
@@ -1810,5 +1776,4 @@
   <child link="wheel_roller3_8_1"/>
   <axis xyz="-0.28033 -0.739199 -0.612372"/>
-  <dynamics damping="0.0"/>
 </joint>
 <joint name="Rev36" type="continuous">
@@ -1817,5 +1782,4 @@
   <child link="wheel_roller3_1_1"/>
   <axis xyz="0.126826 -0.926777 -0.353553"/>
-  <dynamics damping="0.0"/>
 </joint>
 <joint name="Rigid29" type="fixed">
