Commit message: feat: add ball to simulation

File: deepbb_description/urdf/deep_ballbot.xacro (robot description, xacro)
@@ -15,5 +15,5 @@
       <mesh filename="file://$(find deepbb_description)/meshes/base_link.stl" scale="0.001 0.001 0.001"/>
     </geometry>
-    <material name="silver"/>
+    <material name="black"/>
   </visual>
   <collision>
@@ -35,5 +35,5 @@
       <mesh filename="file://$(find deepbb_description)/meshes/base_shell1_1.stl" scale="0.001 0.001 0.001"/>
     </geometry>
-    <material name="silver"/>
+    <material name="white"/>
   </visual>
   <collision>
@@ -55,5 +55,5 @@
       <mesh filename="file://$(find deepbb_description)/meshes/base_shell2_1.stl" scale="0.001 0.001 0.001"/>
     </geometry>
-    <material name="silver"/>
+    <material name="white"/>
   </visual>
   <collision>
@@ -75,5 +75,5 @@
       <mesh filename="file://$(find deepbb_description)/meshes/base_shell3_1.stl" scale="0.001 0.001 0.001"/>
     </geometry>
-    <material name="silver"/>
+    <material name="white"/>
   </visual>
   <collision>
@@ -95,5 +95,5 @@
       <mesh filename="file://$(find deepbb_description)/meshes/base_plate2_1.stl" scale="0.001 0.001 0.001"/>
     </geometry>
-    <material name="silver"/>
+    <material name="grey"/>
   </visual>
   <collision>
@@ -115,5 +115,5 @@
       <mesh filename="file://$(find deepbb_description)/meshes/base_plate3_1.stl" scale="0.001 0.001 0.001"/>
     </geometry>
-    <material name="silver"/>
+    <material name="grey"/>
   </visual>
   <collision>
@@ -135,5 +135,5 @@
       <mesh filename="file://$(find deepbb_description)/meshes/vertical_bay1_1.stl" scale="0.001 0.001 0.001"/>
     </geometry>
-    <material name="silver"/>
+    <material name="grey"/>
   </visual>
   <collision>
@@ -155,5 +155,5 @@
       <mesh filename="file://$(find deepbb_description)/meshes/vertical_bay2_1.stl" scale="0.001 0.001 0.001"/>
     </geometry>
-    <material name="silver"/>
+    <material name="grey"/>
   </visual>
   <collision>
@@ -175,5 +175,5 @@
       <mesh filename="file://$(find deepbb_description)/meshes/vertical_bay3_1.stl" scale="0.001 0.001 0.001"/>
     </geometry>
-    <material name="silver"/>
+    <material name="grey"/>
   </visual>
   <collision>
@@ -195,5 +195,5 @@
       <mesh filename="file://$(find deepbb_description)/meshes/breadboard_1.stl" scale="0.001 0.001 0.001"/>
     </geometry>
-    <material name="silver"/>
+    <material name="white"/>
   </visual>
   <collision>
@@ -215,5 +215,5 @@
       <mesh filename="file://$(find deepbb_description)/meshes/rasbperry_pi_1.stl" scale="0.001 0.001 0.001"/>
     </geometry>
-    <material name="silver"/>
+    <material name="black"/>
   </visual>
   <collision>
@@ -235,5 +235,5 @@
       <mesh filename="file://$(find deepbb_description)/meshes/motor_mount1_1.stl" scale="0.001 0.001 0.001"/>
     </geometry>
-    <material name="silver"/>
+    <material name="grey"/>
   </visual>
   <collision>
@@ -255,5 +255,5 @@
       <mesh filename="file://$(find deepbb_description)/meshes/motor_mount2_1.stl" scale="0.001 0.001 0.001"/>
     </geometry>
-    <material name="silver"/>
+    <material name="grey"/>
   </visual>
   <collision>
@@ -275,5 +275,5 @@
       <mesh filename="file://$(find deepbb_description)/meshes/motor_mount3_1.stl" scale="0.001 0.001 0.001"/>
     </geometry>
-    <material name="silver"/>
+    <material name="grey"/>
   </visual>
   <collision>
@@ -295,5 +295,5 @@
       <mesh filename="file://$(find deepbb_description)/meshes/arduino_mount1_1.stl" scale="0.001 0.001 0.001"/>
     </geometry>
-    <material name="silver"/>
+    <material name="grey"/>
   </visual>
   <collision>
@@ -315,5 +315,5 @@
       <mesh filename="file://$(find deepbb_description)/meshes/arduino_mount2_1.stl" scale="0.001 0.001 0.001"/>
     </geometry>
-    <material name="silver"/>
+    <material name="grey"/>
   </visual>
   <collision>
@@ -335,5 +335,5 @@
       <mesh filename="file://$(find deepbb_description)/meshes/arduino_mount3_1.stl" scale="0.001 0.001 0.001"/>
     </geometry>
-    <material name="silver"/>
+    <material name="grey"/>
   </visual>
   <collision>
@@ -355,5 +355,5 @@
       <mesh filename="file://$(find deepbb_description)/meshes/arduino1_1.stl" scale="0.001 0.001 0.001"/>
     </geometry>
-    <material name="silver"/>
+    <material name="black"/>
   </visual>
   <collision>
@@ -375,5 +375,5 @@
       <mesh filename="file://$(find deepbb_description)/meshes/arduino2_1.stl" scale="0.001 0.001 0.001"/>
     </geometry>
-    <material name="silver"/>
+    <material name="black"/>
   </visual>
   <collision>
@@ -395,5 +395,5 @@
       <mesh filename="file://$(find deepbb_description)/meshes/arduino3_1.stl" scale="0.001 0.001 0.001"/>
     </geometry>
-    <material name="silver"/>
+    <material name="black"/>
   </visual>
   <collision>
@@ -415,5 +415,5 @@
       <mesh filename="file://$(find deepbb_description)/meshes/motor_stator1_1.stl" scale="0.001 0.001 0.001"/>
     </geometry>
-    <material name="silver"/>
+    <material name="black"/>
   </visual>
   <collision>
@@ -435,5 +435,5 @@
       <mesh filename="file://$(find deepbb_description)/meshes/motor_stator2_1.stl" scale="0.001 0.001 0.001"/>
     </geometry>
-    <material name="silver"/>
+    <material name="black"/>
   </visual>
   <collision>
@@ -455,5 +455,5 @@
       <mesh filename="file://$(find deepbb_description)/meshes/motor_stator3_1.stl" scale="0.001 0.001 0.001"/>
     </geometry>
-    <material name="silver"/>
+    <material name="black"/>
   </visual>
   <collision>
@@ -475,5 +475,5 @@
       <mesh filename="file://$(find deepbb_description)/meshes/motor_rotor1_1.stl" scale="0.001 0.001 0.001"/>
     </geometry>
-    <material name="silver"/>
+    <material name="black"/>
   </visual>
   <collision>
@@ -495,5 +495,5 @@
       <mesh filename="file://$(find deepbb_description)/meshes/motor_rotor2_1.stl" scale="0.001 0.001 0.001"/>
     </geometry>
-    <material name="silver"/>
+    <material name="black"/>
   </visual>
   <collision>
@@ -515,5 +515,5 @@
       <mesh filename="file://$(find deepbb_description)/meshes/motor_rotor3_1.stl" scale="0.001 0.001 0.001"/>
     </geometry>
-    <material name="silver"/>
+    <material name="black"/>
   </visual>
   <collision>
@@ -535,5 +535,5 @@
       <mesh filename="file://$(find deepbb_description)/meshes/wheel_body1_1.stl" scale="0.001 0.001 0.001"/>
     </geometry>
-    <material name="silver"/>
+    <material name="white"/>
   </visual>
   <collision>
@@ -555,5 +555,5 @@
       <mesh filename="file://$(find deepbb_description)/meshes/wheel_body2_1.stl" scale="0.001 0.001 0.001"/>
     </geometry>
-    <material name="silver"/>
+    <material name="white"/>
   </visual>
   <collision>
@@ -575,5 +575,5 @@
       <mesh filename="file://$(find deepbb_description)/meshes/wheel_body3_1.stl" scale="0.001 0.001 0.001"/>
     </geometry>
-    <material name="silver"/>
+    <material name="white"/>
   </visual>
   <collision>
@@ -595,5 +595,5 @@
       <mesh filename="file://$(find deepbb_description)/meshes/wheel_roller1_2_1.stl" scale="0.001 0.001 0.001"/>
     </geometry>
-    <material name="silver"/>
+    <material name="grey"/>
   </visual>
   <collision>
@@ -615,5 +615,5 @@
       <mesh filename="file://$(find deepbb_description)/meshes/wheel_roller1_4_1.stl" scale="0.001 0.001 0.001"/>
     </geometry>
-    <material name="silver"/>
+    <material name="grey"/>
   </visual>
   <collision>
@@ -635,5 +635,5 @@
       <mesh filename="file://$(find deepbb_description)/meshes/wheel_roller1_9_1.stl" scale="0.001 0.001 0.001"/>
     </geometry>
-    <material name="silver"/>
+    <material name="grey"/>
   </visual>
   <collision>
@@ -655,5 +655,5 @@
       <mesh filename="file://$(find deepbb_description)/meshes/wheel_roller1_7_1.stl" scale="0.001 0.001 0.001"/>
     </geometry>
-    <material name="silver"/>
+    <material name="grey"/>
   </visual>
   <collision>
@@ -675,5 +675,5 @@
       <mesh filename="file://$(find deepbb_description)/meshes/wheel_roller1_12_1.stl" scale="0.001 0.001 0.001"/>
     </geometry>
-    <material name="silver"/>
+    <material name="grey"/>
   </visual>
   <collision>
@@ -695,5 +695,5 @@
       <mesh filename="file://$(find deepbb_description)/meshes/wheel_roller1_5_1.stl" scale="0.001 0.001 0.001"/>
     </geometry>
-    <material name="silver"/>
+    <material name="grey"/>
   </visual>
   <collision>
@@ -715,5 +715,5 @@
       <mesh filename="file://$(find deepbb_description)/meshes/wheel_roller1_10_1.stl" scale="0.001 0.001 0.001"/>
     </geometry>
-    <material name="silver"/>
+    <material name="grey"/>
   </visual>
   <collision>
@@ -735,5 +735,5 @@
       <mesh filename="file://$(find deepbb_description)/meshes/wheel_roller1_6_1.stl" scale="0.001 0.001 0.001"/>
     </geometry>
-    <material name="silver"/>
+    <material name="grey"/>
   </visual>
   <collision>
@@ -755,5 +755,5 @@
       <mesh filename="file://$(find deepbb_description)/meshes/wheel_roller1_11_1.stl" scale="0.001 0.001 0.001"/>
     </geometry>
-    <material name="silver"/>
+    <material name="grey"/>
   </visual>
   <collision>
@@ -775,5 +775,5 @@
       <mesh filename="file://$(find deepbb_description)/meshes/wheel_roller1_3_1.stl" scale="0.001 0.001 0.001"/>
     </geometry>
-    <material name="silver"/>
+    <material name="grey"/>
   </visual>
   <collision>
@@ -795,5 +795,5 @@
       <mesh filename="file://$(find deepbb_description)/meshes/wheel_roller1_8_1.stl" scale="0.001 0.001 0.001"/>
     </geometry>
-    <material name="silver"/>
+    <material name="grey"/>
   </visual>
   <collision>
@@ -815,5 +815,5 @@
       <mesh filename="file://$(find deepbb_description)/meshes/wheel_roller1_1_1.stl" scale="0.001 0.001 0.001"/>
     </geometry>
-    <material name="silver"/>
+    <material name="grey"/>
   </visual>
   <collision>
@@ -835,5 +835,5 @@
       <mesh filename="file://$(find deepbb_description)/meshes/wheel_roller2_2_1.stl" scale="0.001 0.001 0.001"/>
     </geometry>
-    <material name="silver"/>
+    <material name="grey"/>
   </visual>
   <collision>
@@ -855,5 +855,5 @@
       <mesh filename="file://$(find deepbb_description)/meshes/wheel_roller2_4_1.stl" scale="0.001 0.001 0.001"/>
     </geometry>
-    <material name="silver"/>
+    <material name="grey"/>
   </visual>
   <collision>
@@ -875,5 +875,5 @@
       <mesh filename="file://$(find deepbb_description)/meshes/wheel_roller2_7_1.stl" scale="0.001 0.001 0.001"/>
     </geometry>
-    <material name="silver"/>
+    <material name="grey"/>
   </visual>
   <collision>
@@ -895,5 +895,5 @@
       <mesh filename="file://$(find deepbb_description)/meshes/wheel_roller2_12_1.stl" scale="0.001 0.001 0.001"/>
     </geometry>
-    <material name="silver"/>
+    <material name="grey"/>
   </visual>
   <collision>
@@ -915,5 +915,5 @@
       <mesh filename="file://$(find deepbb_description)/meshes/wheel_roller2_9_1.stl" scale="0.001 0.001 0.001"/>
     </geometry>
-    <material name="silver"/>
+    <material name="grey"/>
   </visual>
   <collision>
@@ -935,5 +935,5 @@
       <mesh filename="file://$(find deepbb_description)/meshes/wheel_roller2_5_1.stl" scale="0.001 0.001 0.001"/>
     </geometry>
-    <material name="silver"/>
+    <material name="grey"/>
   </visual>
   <collision>
@@ -955,5 +955,5 @@
       <mesh filename="file://$(find deepbb_description)/meshes/wheel_roller2_10_1.stl" scale="0.001 0.001 0.001"/>
     </geometry>
-    <material name="silver"/>
+    <material name="grey"/>
   </visual>
   <collision>
@@ -975,5 +975,5 @@
       <mesh filename="file://$(find deepbb_description)/meshes/wheel_roller2_6_1.stl" scale="0.001 0.001 0.001"/>
     </geometry>
-    <material name="silver"/>
+    <material name="grey"/>
   </visual>
   <collision>
@@ -995,5 +995,5 @@
       <mesh filename="file://$(find deepbb_description)/meshes/wheel_roller2_11_1.stl" scale="0.001 0.001 0.001"/>
     </geometry>
-    <material name="silver"/>
+    <material name="grey"/>
   </visual>
   <collision>
@@ -1015,5 +1015,5 @@
       <mesh filename="file://$(find deepbb_description)/meshes/wheel_roller2_3_1.stl" scale="0.001 0.001 0.001"/>
     </geometry>
-    <material name="silver"/>
+    <material name="grey"/>
   </visual>
   <collision>
@@ -1035,5 +1035,5 @@
       <mesh filename="file://$(find deepbb_description)/meshes/wheel_roller2_8_1.stl" scale="0.001 0.001 0.001"/>
     </geometry>
-    <material name="silver"/>
+    <material name="grey"/>
   </visual>
   <collision>
@@ -1055,5 +1055,5 @@
       <mesh filename="file://$(find deepbb_description)/meshes/wheel_roller2_1_1.stl" scale="0.001 0.001 0.001"/>
     </geometry>
-    <material name="silver"/>
+    <material name="grey"/>
   </visual>
   <collision>
@@ -1075,5 +1075,5 @@
       <mesh filename="file://$(find deepbb_description)/meshes/wheel_roller3_2_1.stl" scale="0.001 0.001 0.001"/>
     </geometry>
-    <material name="silver"/>
+    <material name="grey"/>
   </visual>
   <collision>
@@ -1095,5 +1095,5 @@
       <mesh filename="file://$(find deepbb_description)/meshes/wheel_roller3_4_1.stl" scale="0.001 0.001 0.001"/>
     </geometry>
-    <material name="silver"/>
+    <material name="grey"/>
   </visual>
   <collision>
@@ -1115,5 +1115,5 @@
       <mesh filename="file://$(find deepbb_description)/meshes/wheel_roller3_9_1.stl" scale="0.001 0.001 0.001"/>
     </geometry>
-    <material name="silver"/>
+    <material name="grey"/>
   </visual>
   <collision>
@@ -1135,5 +1135,5 @@
       <mesh filename="file://$(find deepbb_description)/meshes/wheel_roller3_7_1.stl" scale="0.001 0.001 0.001"/>
     </geometry>
-    <material name="silver"/>
+    <material name="grey"/>
   </visual>
   <collision>
@@ -1155,5 +1155,5 @@
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
File: deepbb_description/urdf/materials.xacro (robot description, xacro)
@@ -1,6 +1,12 @@
 <?xml version="1.0" ?>
 <robot name="deep_ballbot" xmlns:xacro="http://www.ros.org/wiki/xacro" >
-<material name="silver">
-  <color rgba="0.700 0.700 0.700 1.000"/>
+<material name="black">
+  <color rgba="0.2 0.2 0.2 1.0"/>
+</material>
+<material name="white">
+  <color rgba="1.0 1.0 1.0 1.0"/>
+</material>
+<material name="grey">
+  <color rgba="0.6 0.6 0.6 1.000"/>
 </material>
 </robot>

Commit message: fix: training sim tweaks

File: deepbb_description/urdf/deep_ballbot.xacro (robot description, xacro)
@@ -537,10 +537,4 @@
     <material name="white"/>
   </visual>
-  <collision>
-    <origin rpy="0 0 0" xyz="0.05261 -0.030375 -0.034698"/>
-    <geometry>
-      <mesh filename="file://$(find deepbb_description)/meshes/wheel_body1_1.stl" scale="0.001 0.001 0.001"/>
-    </geometry>
-  </collision>
 </link>
 <link name="wheel_body2_1">
@@ -557,10 +551,4 @@
     <material name="white"/>
   </visual>
-  <collision>
-    <origin rpy="0 0 0" xyz="-0.0 0.060749 -0.034698"/>
-    <geometry>
-      <mesh filename="file://$(find deepbb_description)/meshes/wheel_body2_1.stl" scale="0.001 0.001 0.001"/>
-    </geometry>
-  </collision>
 </link>
 <link name="wheel_body3_1">
@@ -577,10 +565,4 @@
     <material name="white"/>
   </visual>
-  <collision>
-    <origin rpy="0 0 0" xyz="-0.05261 -0.030375 -0.034698"/>
-    <geometry>
-      <mesh filename="file://$(find deepbb_description)/meshes/wheel_body3_1.stl" scale="0.001 0.001 0.001"/>
-    </geometry>
-  </collision>
 </link>
 <link name="wheel_roller1_2_1">

Commit message: fix: switch back to vel control w/ PID inner loop

File: deepbb_description/urdf/deep_ballbot.xacro (robot description, xacro)
@@ -1521,4 +1521,5 @@
   <child link="motor_rotor1_1"/>
   <axis xyz="-0.612372 0.353553 -0.707107"/>
+  <limit effort="500.0" velocity="10.0"/>
 </joint>
 <joint name="MotorJoint2" type="continuous">
@@ -1527,4 +1528,5 @@
   <child link="motor_rotor2_1"/>
   <axis xyz="0.0 -0.707107 -0.707107"/>
+  <limit effort="500.0" velocity="10.0"/>
 </joint>
 <joint name="MotorJoint3" type="continuous">
@@ -1533,4 +1535,5 @@
   <child link="motor_rotor3_1"/>
   <axis xyz="0.612372 0.353553 -0.707107"/>
+  <limit effort="500.0" velocity="10.0"/>
 </joint>
 <joint name="Rigid26" type="fixed">

Commit message: logs + changes to training

File: deepbb_description/urdf/deep_ballbot.xacro (robot description, xacro)
@@ -1521,5 +1521,5 @@
   <child link="motor_rotor1_1"/>
   <axis xyz="-0.612372 0.353553 -0.707107"/>
-  <limit effort="500.0" velocity="10.0"/>
+  <limit effort="500.0" velocity="20.0"/>
 </joint>
 <joint name="MotorJoint2" type="continuous">
@@ -1528,5 +1528,5 @@
   <child link="motor_rotor2_1"/>
   <axis xyz="0.0 -0.707107 -0.707107"/>
-  <limit effort="500.0" velocity="10.0"/>
+  <limit effort="500.0" velocity="20.0"/>
 </joint>
 <joint name="MotorJoint3" type="continuous">
@@ -1535,5 +1535,5 @@
   <child link="motor_rotor3_1"/>
   <axis xyz="0.612372 0.353553 -0.707107"/>
-  <limit effort="500.0" velocity="10.0"/>
+  <limit effort="500.0" velocity="20.0"/>
 </joint>
 <joint name="Rigid26" type="fixed">
